File: PCB/xESC/xESC.kicad_pcb (KiCad board)
At the start: 2 copper layers, 24 parts, among them Q1 BSC440N10NS3G, Q2 BSC440N10NS3G, Q3 BSC440N10NS3G, Q4 BSC440N10NS3G, Q5 BSC440N10NS3G, Q6 BSC440N10NS3G, U1 ATmega328-AU, U2 TMC6100-LA, U3 LMV321, U4 MIC5504-1.8YM5

Commit message: wip
Parts:
- added D1: LED, LED_SMD:LED_0805_2012Metric_Pad1.15x1.40mm_HandSolder, F.Cu at (226.1, 163.8)
- added JP8: SolderJumper_2_Open, Jumper:SolderJumper-2_P1.3mm_Open_Pad1.0x1.5mm, F.Cu at (249.4, 159.4)
- added R10: R, Resistor_SMD:R_0805_2012Metric, F.Cu at (236.1, 159.1)
- added R11: R, Resistor_SMD:R_0805_2012Metric, F.Cu at (235.0, 162.1)
- added R8: 10kR, Resistor_SMD:R_0805_2012Metric, F.Cu at (231.7, 159.1)
- added R9: 150R, Resistor_SMD:R_0805_2012Metric, F.Cu at (230.6, 163.8)
- added Y1: Resonator, Crystal:Resonator_SMD_muRata_CSTxExxV-3Pin_3.0x1.1mm_HandSoldering, F.Cu at (245.1, 160.1)
- moved U3 42.1 mm to (226.5, 160.0)
Connections:
- U1 pad 20: (no net) -> Net-(C14-Pad1)
- U1 pad 7: (no net) -> Net-(U1-Pad7)
- U1 pad 8: (no net) -> Net-(U1-Pad8)
- U2 pad 10: (no net) -> /Power/SS
- U2 pad 22: (no net) -> /Power/VCC_IO
- U2 pad 23: (no net) -> /Power/FAULT
- U2 pad 3: (no net) -> /Power/LS_W
- U2 pad 31: (no net) -> /Power/HS_W
- U2 pad 32: (no net) -> /Power/W
- U2 pad 33: (no net) -> /Power/V
- U2 pad 34: (no net) -> /Power/HS_V
- U2 pad 36: (no net) -> /Power/LS_U
- U2 pad 37: (no net) -> /Power/HS_U
- U2 pad 4: (no net) -> /Power/LS_V
- U2 pad 5: (no net) -> /Power/LS_U
- U3 pad 1: (no net) -> /Power/BridgeMosfets/GND
- U3 pad 2: (no net) -> GND
- U3 pad 3: (no net) -> Net-(R10-Pad1)
- U3 pad 4: (no net) -> /Power/I_SENSE
- U3 pad 5: (no net) -> /Power/VCC_IO

Commit message: wip
Parts:
- added C1: 100nF, Capacitor_SMD:C_0805_2012Metric_Pad1.18x1.45mm_HandSolder, F.Cu at (217.4, 149.8)
- added C10: CP, Capacitor_THT:CP_Radial_D8.0mm_P3.50mm, F.Cu at (153.0, 76.0)
- added C11: 470nF, Capacitor_SMD:C_0805_2012Metric_Pad1.18x1.45mm_HandSolder, F.Cu at (193.6, 154.8)
- added C12: 4.7uF, Capacitor_SMD:C_0805_2012Metric_Pad1.18x1.45mm_HandSolder, F.Cu at (205.1, 153.8)
- added C13: 2.2uF, Capacitor_SMD:C_0805_2012Metric_Pad1.18x1.45mm_HandSolder, F.Cu at (212.6, 143.8)
- added C14: 100nF, Capacitor_SMD:C_0805_2012Metric_Pad1.18x1.45mm_HandSolder, F.Cu at (237.0, 143.8)
- added C15: 10pF, Capacitor_SMD:C_0805_2012Metric_Pad1.18x1.45mm_HandSolder, F.Cu at (226.6, 153.3)
- added C16: 10pF, Capacitor_SMD:C_0805_2012Metric_Pad1.18x1.45mm_HandSolder, F.Cu at (231.4, 147.3)
- added C17: 10pF, Capacitor_SMD:C_0805_2012Metric_Pad1.18x1.45mm_HandSolder, F.Cu at (226.6, 150.3)
- added C18: 100nF, Capacitor_SMD:C_0805_2012Metric_Pad1.18x1.45mm_HandSolder, F.Cu at (232.2, 143.8)
- added C19: 100nF, Capacitor_SMD:C_0805_2012Metric_Pad1.18x1.45mm_HandSolder, F.Cu at (226.6, 147.3)
- added C2: c?, Capacitor_SMD:C_0805_2012Metric_Pad1.18x1.45mm_HandSolder, F.Cu at (214.7, 152.8)
- added C20: CP, Capacitor_THT:CP_Radial_D8.0mm_P3.50mm, F.Cu at (153.0, 87.0)
- added C3: c?, Capacitor_SMD:C_0805_2012Metric_Pad1.18x1.45mm_HandSolder, F.Cu at (209.9, 156.8)
- added C4: 100nF, Capacitor_SMD:C_0805_2012Metric_Pad1.18x1.45mm_HandSolder, F.Cu at (217.4, 146.8)
- added C5: c?, Capacitor_SMD:C_0805_2012Metric_Pad1.18x1.45mm_HandSolder, F.Cu at (212.6, 149.8)
- added C6: 100nF@16V, Capacitor_SMD:C_0805_2012Metric_Pad1.18x1.45mm_HandSolder, F.Cu at (209.9, 153.8)
- added C7: 100nF, Capacitor_SMD:C_0805_2012Metric_Pad1.18x1.45mm_HandSolder, F.Cu at (205.1, 156.8)
- added C8: 100nF, Capacitor_SMD:C_0805_2012Metric_Pad1.18x1.45mm_HandSolder, F.Cu at (217.4, 143.8)
- added C9: 22n@100V, Capacitor_SMD:C_0805_2012Metric_Pad1.18x1.45mm_HandSolder, F.Cu at (212.6, 146.8)
- added D2: D_Schottky, Diode_SMD:D_0805_2012Metric_Pad1.15x1.40mm_HandSolder, F.Cu at (241.8, 143.8)
- added D3: D_Schottky, Diode_SMD:D_0805_2012Metric_Pad1.15x1.40mm_HandSolder, F.Cu at (236.2, 146.8)
- added D4: D_Schottky, Diode_SMD:D_0805_2012Metric_Pad1.15x1.40mm_HandSolder, F.Cu at (231.4, 150.4)
- added JP9: SolderJumper_3_Bridged12, Jumper:SolderJumper-3_P1.3mm_Bridged12_Pad1.0x1.5mm_NumberLabels, F.Cu at (227.0, 144.1)
- added R12: 1kR, Resistor_SMD:R_0805_2012Metric, F.Cu at (236.0, 153.3)
- added R13: 1kR, Resistor_SMD:R_0805_2012Metric, F.Cu at (240.8, 146.8)
- added R14: 1kR, Resistor_SMD:R_0805_2012Metric, F.Cu at (236.0, 150.3)
- added R15: 10kR, Resistor_SMD:R_0805_2012Metric, F.Cu at (231.2, 153.3)
- added R16: 1kR, Resistor_SMD:R_0805_2012Metric_Pad1.20x1.40mm_HandSolder, F.Cu at (194.4, 163.1)
- JP2, JP3, JP4, JP5, JP6, JP7, R1, R2, R3, R4, R5, R6, R7: moved to B.Cu
- moved U2 120.6 mm to (137.8, 78.0), turned to 225 degrees
- moved JP6 118.1 mm to (141.0, 95.0), turned to 90 degrees
- moved R5 107.1 mm to (139.0, 95.0), turned to 270 degrees
- moved JP2 103.6 mm to (132.0, 86.8), turned to 90 degrees
- moved JP4 103.4 mm to (142.5, 86.5), turned to 90 degrees
- moved R7 102.7 mm to (160.0, 82.0), turned to 180 degrees
- moved R1 101.3 mm to (130.0, 86.8), turned to 270 degrees
- moved JP7 96.7 mm to (168.0, 72.5), turned to 270 degrees
- moved R6 94.7 mm to (165.8, 72.5), turned to 90 degrees
- moved R3 93.5 mm to (140.5, 86.5), turned to 270 degrees
- moved Q6 91.5 mm to (165.0, 91.0), turned to 90 degrees
- moved JP5 90.7 mm to (163.5, 72.5), turned to 270 degrees
- moved Q5 89.4 mm to (159.0, 91.0), turned to 270 degrees
- moved JP3 89.3 mm to (159.0, 72.5), turned to 270 degrees
- moved R4 88.9 mm to (161.2, 72.5), turned to 90 degrees
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Connections:
- net /Power/5V renamed /5V
- net /Power/V renamed /PHASE_V
- net /Power/V_M renamed /V_M
- net /Power/W renamed /PHASE_W
- JP1 pad 2: /Power/VCC_IO -> VCC
- Q1 pad 1: /Power/LS_U -> /PHASE_U
- Q1 pad 2: /Power/LS_U -> /PHASE_U
- Q1 pad 3: /Power/LS_U -> /PHASE_U
- Q2 pad 5: /Power/LS_U -> /PHASE_U
- R11 pad 1: /Power/I_SENSE -> /I_SENSE
- R8 pad 1: /Power/VCC_IO -> VCC
- R8 pad 2: /Power/SS -> /DRV_SS
- R9 pad 1: /Power/FAULT -> /FAULT
- U1 pad 1: (no net) -> /U_ENABLE
- U1 pad 10: (no net) -> /W_ENABLE
- U1 pad 11: (no net) -> /W_DIR
- U1 pad 12: (no net) -> /FAULT
- U1 pad 13: (no net) -> /INPUT
- U1 pad 15: (no net) -> /MOSI
- U1 pad 16: (no net) -> /MISO
- U1 pad 17: (no net) -> /SCK
- U1 pad 19: (no net) -> /INPUT
- U1 pad 2: (no net) -> /V_DIR
- U1 pad 23: (no net) -> /HALL_U
- U1 pad 24: (no net) -> /HALL_V
- U1 pad 25: (no net) -> /HALL_W
- U1 pad 26: (no net) -> /I_SENSE
- U1 pad 27: (no net) -> /DRV_ENABLE
- U1 pad 28: (no net) -> /DRV_SS
- U1 pad 29: (no net) -> /RESET
- U1 pad 31: (no net) -> /TXD
- U1 pad 32: (no net) -> /U_DIR
- U1 pad 9: (no net) -> /V_ENABLE
- U2 pad 1: (no net) -> Net-(C2-Pad1)
- U2 pad 10: /Power/SS -> /DRV_SS
- U2 pad 11: (no net) -> /SCK
- U2 pad 12: (no net) -> /MOSI
- U2 pad 13: (no net) -> /MISO
- U2 pad 14: (no net) -> /U_DIR
- U2 pad 15: (no net) -> /U_ENABLE
- U2 pad 16: /Power/VCC_IO -> VCC
- U2 pad 17: (no net) -> /V_DIR
- U2 pad 18: (no net) -> /V_ENABLE
- U2 pad 19: (no net) -> /W_DIR
- U2 pad 20: (no net) -> /W_ENABLE
- U2 pad 22: /Power/VCC_IO -> VCC
- U2 pad 23: /Power/FAULT -> /FAULT
- U2 pad 24: (no net) -> /DRV_ENABLE
- U2 pad 26: (no net) -> Net-(C9-Pad2)
- U2 pad 27: (no net) -> Net-(C9-Pad1)
- U2 pad 29: (no net) -> Net-(C6-Pad1)
- U2 pad 30: (no net) -> Net-(C5-Pad1)
- U2 pad 35: (no net) -> Net-(C3-Pad1)
- U2 pad 36: /Power/LS_U -> /PHASE_U
- U2 pad 6: (no net) -> Net-(C12-Pad1)
- U3 pad 4: /Power/I_SENSE -> /I_SENSE
- U3 pad 5: /Power/VCC_IO -> VCC
Routing:
- net Net-(JP7-Pad2): track 0.00 -> 28.2 mm, vias 0 -> 1
- net Net-(JP5-Pad2): track 0.00 -> 22.8 mm, vias 0 -> 1
- net Net-(JP3-Pad2): track 0.00 -> 17.8 mm, vias 0 -> 1
- net /Power/LS_U: track 0.00 -> 2.42 mm
- net /Power/LS_W: track 0.00 -> 2.36 mm
- net /Power/LS_V: track 0.00 -> 2.36 mm
- net Net-(JP6-Pad2): track 0.00 -> 2.11 mm
- net Net-(JP4-Pad2): track 0.00 -> 2.11 mm
- net Net-(JP2-Pad2): track 0.00 -> 2.11 mm
- net /Power/HS_W: track 0.00 -> 2.11 mm
- net /Power/HS_V: track 0.00 -> 2.11 mm
- net /Power/HS_U: track 0.00 -> 2.11 mm
- net /Power/BridgeMosfets/GND: vias 0 -> 33
- added copper zone on F.Cu, net /PHASE_U
- added copper zone on F.Cu, net /PHASE_V
- added copper zone on F.Cu, net /PHASE_W
- added copper zone on B.Cu, net /Power/BridgeMosfets/GND
- added copper zone on F.Cu, net /Power/BridgeMosfets/GND
- added copper zone on F.Cu, net /V_M
- added copper zone on F.Cu, net GND
Other:
- net class Default: clearance 0.2 -> 0.127; trace_width 0.25 -> 0.127; via_dia 0.8 -> 0.6; via_drill 0.4 -> 0.3
- rule trace_clearance: 0.2 -> 0.127
- rule trace_min: 0.2 -> 0.127
- rule via_min_size: 0.4 -> 0.6

Commit message: wip
Parts:
- removed JP8: SolderJumper_2_Open, Jumper:SolderJumper-2_P1.3mm_Open_Pad1.0x1.5mm
- added J1: Conn_01x05_Male, Connector_PinHeader_2.54mm:PinHeader_1x05_P2.54mm_Vertical, F.Cu at (216.1, 56.6)
- added J2: Conn_01x03_Male, Connector_PinHeader_2.54mm:PinHeader_1x03_P2.54mm_Vertical, F.Cu at (250.1, 28.7)
- added J3: Conn_01x03_Male, Connector_PinHeader_2.54mm:PinHeader_1x03_P2.54mm_Vertical, F.Cu at (250.1, 24.7)
- added R17: 1kR, Resistor_SMD:R_0805_2012Metric_Pad1.20x1.40mm_HandSolder, F.Cu at (240.8, 28.7)
- added R18: 1kR, Resistor_SMD:R_0805_2012Metric_Pad1.20x1.40mm_HandSolder, F.Cu at (240.8, 24.7)
- R7: moved to F.Cu
- U1: moved to B.Cu
- moved Y1 140.3 mm to (223.5, 21.5), turned to 270 degrees
- moved R10 129.2 mm to (191.0, 38.0), turned to 90 degrees
- moved R11 127.9 mm to (191.0, 42.0), turned to 270 degrees
- moved C18 126.6 mm to (223.5, 17.5), turned to 90 degrees
- moved U3 124.2 mm to (187.8, 42.0), turned to 90 degrees
- moved C3 123.3 mm to (187.8, 35.5)
- moved C11 122.1 mm to (176.0, 34.0), turned to 90 degrees
- moved C19 121.9 mm to (223.5, 25.5), turned to 90 degrees
- moved R8 121.8 mm to (198.2, 42.0), turned to 270 degrees
- moved R9 120.3 mm to (188.2, 51.2), turned to 270 degrees
- moved D1 119.5 mm to (186.0, 51.2), turned to 270 degrees
- moved C5 119.4 mm to (187.8, 33.0)
- moved C2 117.9 mm to (187.8, 38.0)
- moved C8 113.7 mm to (194.2, 32.5)
- moved C12 111.1 mm to (194.2, 43.2)
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Connections:
- JP4 pad 1: /Power/HS_V -> /Power/HS_W
- JP5 pad 1: /Power/LS_V -> /Power/LS_W
- JP6 pad 1: /Power/HS_W -> /Power/HS_V
- JP7 pad 1: /Power/LS_W -> /Power/LS_V
- Q3 pad 1: /PHASE_V -> /PHASE_W
- Q3 pad 2: /PHASE_V -> /PHASE_W
- Q3 pad 3: /PHASE_V -> /PHASE_W
- Q4 pad 5: /PHASE_V -> /PHASE_W
- Q5 pad 1: /PHASE_W -> /PHASE_V
- Q5 pad 2: /PHASE_W -> /PHASE_V
- Q5 pad 3: /PHASE_W -> /PHASE_V
- Q6 pad 5: /PHASE_W -> /PHASE_V
- R3 pad 2: /Power/HS_V -> /Power/HS_W
- R4 pad 2: /Power/LS_V -> /Power/LS_W
- R5 pad 2: /Power/HS_W -> /Power/HS_V
- R6 pad 2: /Power/LS_W -> /Power/LS_V
- U1 pad 13: /INPUT -> /INPUT_PWM
- U1 pad 19: /INPUT -> /INPUT_ANALOG
Routing:
- net /PHASE_U: track 0.00 -> 59.0 mm, vias 0 -> 19
- net /PHASE_V: track 0.00 -> 57.4 mm, vias 0 -> 19
- net /PHASE_W: track 0.00 -> 45.2 mm, vias 0 -> 18
- net /Power/HS_U: track 2.11 -> 43.9 mm, vias 0 -> 1
- net Net-(JP4-Pad2): track 2.11 -> 37.2 mm, vias 0 -> 1
- net VCC: track 0.00 -> 33.7 mm, vias 0 -> 2
- net /Power/HS_V: track 2.11 -> 33.2 mm, vias 0 -> 1
- net Net-(JP6-Pad2): track 2.11 -> 32.7 mm, vias 0 -> 1
- net /Power/HS_W: track 2.11 -> 30.1 mm, vias 0 -> 1
- net /Power/LS_U: track 2.42 -> 27.0 mm, vias 0 -> 1
- net Net-(JP2-Pad2): track 2.11 -> 26.5 mm, vias 0 -> 1
- net Net-(C9-Pad1): track 0.00 -> 22.2 mm, vias 0 -> 1
- net /Power/LS_V: track 2.36 -> 20.1 mm, vias 0 -> 1
- net Net-(JP9-Pad2): track 0.00 -> 16.6 mm, vias 0 -> 3
- net /Power/BridgeMosfets/GND: track 0.00 -> 14.4 mm, vias 33 -> 1
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- added copper zone on F.Cu, net /5V
- added copper zone on F.Cu, net /HALL_U
- added copper zone on F.Cu, net /HALL_V
- added copper zone on F.Cu, net /HALL_W
- added copper zone on B.Cu, net /PHASE_U
- added copper zone on B.Cu, net /PHASE_V
- added copper zone on B.Cu, net /PHASE_W
- added copper zone on B.Cu, net /V_M
- added copper zone on B.Cu, net GND
- removed copper zone on B.Cu, net /Power/BridgeMosfets/GND
Other:
- board outline added: 65 x 28 mm
- net class Default: clearance 0.127 -> 0.2; trace_width 0.127 -> 0.2
- rule trace_clearance: 0.127 -> 0.2
- rule trace_min: 0.127 -> 0.2

Commit message: wip
Parts:
- removed C8: 100nF, Capacitor_SMD:C_0805_2012Metric_Pad1.18x1.45mm_HandSolder
- removed D3, D4: D_Schottky, Diode_SMD:D_0805_2012Metric_Pad1.15x1.40mm_HandSolder
- removed JP1, JP9: SolderJumper_3_Bridged12, Jumper:SolderJumper-3_P1.3mm_Bridged12_Pad1.0x1.5mm_NumberLabels
- removed U4: MIC5504-1.8YM5, Package_TO_SOT_SMD:SOT-23-5_HandSoldering
- added H1: MountingHole_Pad, MountingHole:MountingHole_2.2mm_M2_DIN965_Pad, F.Cu at (158.0, 32.8)
- added H2: MountingHole_Pad, MountingHole:MountingHole_2.2mm_M2_DIN965_Pad, F.Cu at (211.5, 32.8)
- added H3: MountingHole_Pad, MountingHole:MountingHole_2.2mm_M2_DIN965_Pad, F.Cu at (211.5, 57.2)
- added H4: MountingHole_Pad, MountingHole:MountingHole_2.2mm_M2_DIN965_Pad, F.Cu at (158.0, 57.2)
- added J4: Conn_01x03_Male, Connector_PinHeader_2.54mm:PinHeader_1x03_P2.54mm_Vertical, F.Cu at (207.5, 34.3)
- added TP1: TestPoint, xESC:TestPoint_Pad_1.5x1.5mm, F.Cu at (204.9, 32.0)
- added TP2: TestPoint, xESC:TestPoint_Pad_1.5x1.5mm, F.Cu at (202.4, 32.0)
- added TP3: TestPoint, xESC:TestPoint_Pad_1.5x1.5mm, B.Cu at (205.0, 32.0)
- added TP4: TestPoint, xESC:TestPoint_Pad_1.5x1.5mm, B.Cu at (199.9, 32.0)
- added TP5: TestPoint, xESC:TestPoint_Pad_1.5x1.5mm, B.Cu at (202.4, 32.0)
- added TP6: TestPoint, xESC:TestPoint_Pad_1.5x1.5mm, B.Cu at (192.2, 32.0)
- added TP7: TestPoint, xESC:TestPoint_Pad_1.5x1.5mm, F.Cu at (207.5, 32.0)
- added TP8: TestPoint, xESC:TestPoint_Pad_1.5x1.5mm, B.Cu at (197.3, 32.0)
- added TP9: TestPoint, xESC:TestPoint_Pad_1.5x1.5mm, B.Cu at (194.8, 32.0)
- C15, C16, C17, D2, Q2, Q4, Q6, R10, R11, R12, R13, R14, R15, R17, R18, R7, R8, U3: moved to B.Cu
- JP2, JP3, JP4, JP5, JP6, JP7, R1, R2, R3, R4, R5, R6, U1: moved to F.Cu
- moved R15 77.1 mm to (188.4, 32.0)
- moved R16 56.4 mm to (199.6, 33.6), turned to 90 degrees
- moved J3 48.3 mm to (203.5, 37.4), turned to 90 degrees
- moved J2 47.9 mm to (203.5, 39.9), turned to 90 degrees
- moved R18 43.3 mm to (199.5, 37.5)
- moved R17 42.9 mm to (199.5, 40.0)
- moved Y1 40.7 mm to (184.5, 33.0), turned to 0 degrees
- moved C18 38.1 mm to (188.5, 32.5), turned to 0 degrees
- moved C10 32.8 mm to (171.5, 49.5), turned to 0 degrees
- moved C19 29.7 mm to (202.2, 46.2), turned to 180 degrees
- moved C20 28.8 mm to (171.5, 40.5), turned to 0 degrees
- moved C5 28.2 mm to (202.2, 57.2), turned to 180 degrees
- moved C3 24.3 mm to (202.2, 55.0), turned to 180 degrees
- moved D2 23.9 mm to (188.4, 34.2)
- moved C2 20.7 mm to (202.2, 52.8), turned to 180 degrees
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Connections:
- C13 pad 1: /5V -> VCC
- D2 pad 2: /HALL_W -> Net-(D2-Pad2)
- J1 pad 5: /5V -> VCC
- R12 pad 1: Net-(JP9-Pad2) -> VCC
- R13 pad 1: Net-(JP9-Pad2) -> VCC
- R14 pad 1: Net-(JP9-Pad2) -> VCC
- R16 pad 1: (no net) -> Net-(J4-Pad3)
- U1 pad 14: (no net) -> /EXT_SPI_SS
- U1 pad 30: (no net) -> /RXD
- U2 pad 7: /5V -> VCC
Routing:
- net VCC: track 33.7 -> 104.8 mm, vias 2 -> 11
- net /V_M: track 0.00 -> 60.4 mm, vias 8 -> 45
- net /MISO: track 0.00 -> 30.2 mm, vias 0 -> 1
- net /SCK: track 0.00 -> 29.2 mm, vias 0 -> 1
- net /MOSI: track 0.00 -> 29.1 mm, vias 0 -> 2
- net /DRV_ENABLE: track 0.00 -> 27.9 mm, vias 0 -> 2
- net GND: track 0.00 -> 25.1 mm, vias 49 -> 72
- net /INPUT_PWM: track 0.00 -> 24.7 mm, vias 0 -> 2
- net /I_SENSE: track 0.00 -> 23.7 mm, vias 0 -> 1
- net /EXT_SPI_SS: track 0.00 -> 21.1 mm, vias 0 -> 1
- net /INPUT_ANALOG: track 0.00 -> 19.5 mm, vias 0 -> 2
- net /DRV_SS: track 0.00 -> 19.4 mm, vias 0 -> 3
- net /V_DIR: track 0.00 -> 19.0 mm, vias 0 -> 2
- net /U_ENABLE: track 0.00 -> 17.4 mm, vias 0 -> 2
- net Net-(JP9-Pad2): track 16.6 -> 0.00 mm, vias 3 -> 0
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- added copper zone on B.Cu, net /EXT_SPI_SS
- added copper zone on F.Cu, net /INPUT_ANALOG
- added copper zone on F.Cu, net /INPUT_PWM
- added copper zone on B.Cu, net /MISO
- added copper zone on B.Cu, net /MOSI
- added copper zone on B.Cu, net /Power/BridgeMosfets/GND
- added copper zone on B.Cu, net /RESET
- added copper zone on F.Cu, net /RXD
- added copper zone on B.Cu, net /SCK
- added copper zone on B.Cu, net Net-(D2-Pad2)
- added copper zone on F.Cu, net Net-(J4-Pad3)
- added copper zone on F.Cu, net VCC
- removed copper zone on F.Cu, net /5V
- removed copper zone on F.Cu, net /Power/BridgeMosfets/GND
Other:
- board size 65 x 28 mm -> 58 x 29 mm
- board text added: "+"
- board text added: "-"
- board text added: "5V"
- board text added: "AIN"
- board text added: "GND"
- board text added: "PWM"
- board text added: "U"
- board text added: "V"
- board text added: "V+"
- board text added: "W"
