File: PCB/xESC/xESC.kicad_pcb (KiCad board)
At the start: 2 copper layers, 58 x 29 mm, 72 parts, among them J1 Conn_01x05_Male, J2 Conn_01x03_Male, J3 Conn_01x03_Male, J4 Conn_01x03_Male, Q1 BSC440N10NS3G, Q2 BSC440N10NS3G, Q3 BSC440N10NS3G, Q4 BSC440N10NS3G, Q5 BSC440N10NS3G, Q6 BSC440N10NS3G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

Commit message: added logo, version and github link
Parts:
- added G***: LOGO, x-tech-logo:x-tech-logo, B.Cu at (190.5, 52.0)
- added REF**: ESD-Logo_6.6x6mm_SilkScreen, Symbol:ESD-Logo_6.6x6mm_SilkScreen, B.Cu at (183.5, 51.8)
Other:
- board text added: "v1.0 - License CC BY-NC-SA 4.0 https://github.com/ClemensElflein/xESC"
