File: PCB/xESC2/xESC2.kicad_pcb (KiCad board)
At the start: 2 copper layers, 32.9 x 34.4 mm, 24 parts, among them Q1 BSC026N08NS5, Q2 BSC026N08NS5, Q3 BSC026N08NS5, Q4 BSC026N08NS5, Q5 BSC026N08NS5, Q6 BSC026N08NS5

Commit message: power schematic wip
Parts:
- added C10: 470nF/16V, Capacitor_SMD:C_0603_1608Metric, F.Cu at (139.6, 105.1)
- added C11: 22nF/100V, Capacitor_SMD:C_0603_1608Metric, F.Cu at (143.6, 102.6)
- added C12: 100nF/100V, Capacitor_SMD:C_0805_2012Metric, F.Cu at (139.8, 96.8)
- added C13: 100nF/100V, Capacitor_SMD:C_0805_2012Metric, F.Cu at (135.4, 102.8)
- added C14: 100nF/100V, Capacitor_SMD:C_0805_2012Metric, F.Cu at (139.8, 99.8)
- added C4: 2.2uF/50V, Capacitor_SMD:C_0805_2012Metric, F.Cu at (135.4, 96.8)
- added C5: 2.2uF/50V, Capacitor_SMD:C_0805_2012Metric, F.Cu at (135.4, 99.8)
- added C6: 100nF/50V, Capacitor_SMD:C_0603_1608Metric, F.Cu at (144.1, 96.5)
- added C7: 100nF/50V, Capacitor_SMD:C_0603_1608Metric, F.Cu at (139.6, 102.6)
- added C8: 470nF/16V, Capacitor_SMD:C_0603_1608Metric, F.Cu at (144.1, 99.1)
- added C9: 470nF/16V, Capacitor_SMD:C_0603_1608Metric, F.Cu at (148.1, 96.5)
- added R13: DNP, Resistor_SMD:R_0603_1608Metric, F.Cu at (148.1, 99.1)
- added R14: DNP, Resistor_SMD:R_0603_1608Metric, F.Cu at (143.6, 105.1)
- added R15: DNP, Resistor_SMD:R_0603_1608Metric, F.Cu at (147.7, 101.6)
- added U1: TMC6200-TA, footprints:TMC6200-TA, F.Cu at (95.8, 83.2)
- moved Q4 44.1 mm to (108.0, 98.6)
- moved R5 40.0 mm to (120.1, 100.8)
- moved Q6 36.9 mm to (135.9, 81.6)
- moved R6 34.2 mm to (120.1, 98.3)
- moved R7 34.2 mm to (108.2, 92.8)
- moved TP2 34.2 mm to (115.1, 100.1)
- moved C2 34.2 mm to (123.6, 92.0)
- moved R8 28.7 mm to (122.8, 95.0)
- moved R10 27.4 mm to (148.1, 81.3)
- moved R9 27.4 mm to (150.7, 77.9)
- moved C3 27.4 mm to (151.5, 75.0)
- moved R11 27.4 mm to (136.1, 75.8)
- moved R12 27.4 mm to (148.1, 83.8)
- moved TP3 27.4 mm to (143.0, 83.1)
- moved Q3 24.4 mm to (116.7, 93.7)
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Connections:
- net /Power/MOSFET/DRV renamed /Power/DRV_U
- net /Power/sheet61A57DC9/DRV renamed /Power/DRV_V
- net /Power/sheet61A580CB/DRV renamed /Power/DRV_W
- C1 pad 1: /Power/MOSFET/VM -> /Power/VM
- C2 pad 1: /Power/sheet61A57DC9/VM -> /Power/VM
- C3 pad 1: /Power/sheet61A580CB/VM -> /Power/VM
- Q1 pad 5: /Power/MOSFET/VM -> /Power/VM
- Q3 pad 5: /Power/sheet61A57DC9/VM -> /Power/VM
- Q5 pad 5: /Power/sheet61A580CB/VM -> /Power/VM
- R1 pad 2: (no net) -> /Power/HSU
- R10 pad 2: (no net) -> /Power/LSW
- R12 pad 2: (no net) -> /Power/SENSE_W
- R2 pad 2: (no net) -> /Power/LSU
- R4 pad 2: (no net) -> /Power/SENSE_U
- R5 pad 2: (no net) -> /Power/HSV
- R6 pad 2: (no net) -> /Power/LSV
- R8 pad 2: (no net) -> /Power/SENSE_V
- R9 pad 2: (no net) -> /Power/HSW

Commit message: wip
Parts:
- added C15: 1uF/50V, Capacitor_SMD:C_0805_2012Metric, F.Cu at (145.5, 74.5)
- added C16: 1uF/50V, Capacitor_SMD:C_0805_2012Metric, F.Cu at (141.0, 74.5)
- added C17: 1uF/50V, Capacitor_SMD:C_0805_2012Metric, F.Cu at (150.0, 99.0)
- added C18: 100uF/16V, Capacitor_SMD:CP_Elec_6.3x7.7, F.Cu at (150.0, 80.0)
- added C19: 10uF/25V, Capacitor_SMD:C_1206_3216Metric, F.Cu at (158.0, 70.5)
- added C20: 10uF/25V, Capacitor_SMD:C_1206_3216Metric, F.Cu at (161.5, 70.5)
- added C21: 47uF/100V, Capacitor_THT:CP_Radial_D8.0mm_P3.50mm, F.Cu at (142.5, 70.0)
- added C22: 220uF/63V, Capacitor_THT:CP_Radial_D10.0mm_P5.00mm_P7.50mm, F.Cu at (171.5, 98.0)
- added C23: 220uF/63V, Capacitor_THT:CP_Radial_D10.0mm_P5.00mm_P7.50mm, F.Cu at (171.5, 69.0)
- added C24: 1nF/100V, Capacitor_SMD:C_0603_1608Metric, F.Cu at (197.5, 78.0)
- added C25: 1nF/100V, Capacitor_SMD:C_0603_1608Metric, F.Cu at (197.5, 89.5)
- added C26: 1nF/100V, Capacitor_SMD:C_0603_1608Metric, F.Cu at (197.5, 101.0)
- added D1: SS36, Diode_SMD:D_SMA, F.Cu at (143.0, 99.0)
- added D2: LED, LED_SMD:LED_0603_1608Metric, F.Cu at (157.5, 90.0)
- added H1: MountingHole_Pad, MountingHole:MountingHole_2.7mm_M2.5_DIN965_Pad, F.Cu at (203.5, 65.5)
- added H2: MountingHole_Pad, MountingHole:MountingHole_2.7mm_M2.5_DIN965_Pad, F.Cu at (203.5, 101.5)
- added H3: MountingHole_Pad, MountingHole:MountingHole_2.7mm_M2.5_DIN965_Pad, F.Cu at (268.2, 87.5)
- added H4: MountingHole_Pad, MountingHole:MountingHole_2.7mm_M2.5_DIN965_Pad, F.Cu at (268.2, 93.8)
- added L1: 47uH/3A, Inductor_SMD:L_Wuerth_HCI-1040, F.Cu at (145.5, 91.0)
- added R16: 150R, Resistor_SMD:R_0603_1608Metric, F.Cu at (159.5, 90.0)
- added TP4: TestPoint, TestPoint:TestPoint_Pad_4.0x4.0mm, F.Cu at (178.0, 65.0)
- added TP5: TestPoint, TestPoint:TestPoint_Pad_4.0x4.0mm, F.Cu at (178.0, 101.5)
- added TP6: TestPoint, TestPoint:TestPoint_Pad_4.0x4.0mm, F.Cu at (159.5, 65.0)
- added TP7: TestPoint, TestPoint:TestPoint_Pad_4.0x4.0mm, F.Cu at (159.5, 101.5)
- added U2: XL2001, Package_SO:SOP-8_3.9x4.9mm_P1.27mm, F.Cu at (141.0, 80.0)
- added U3: AMS1117-3.3, Package_TO_SOT_SMD:SOT-223-3_TabPin2, F.Cu at (152.0, 68.5)
- moved TP2 89.9 mm to (203.5, 83.5), turned to 90 degrees
- moved R7 89.8 mm to (197.5, 83.5), turned to 90 degrees
- moved R3 89.4 mm to (197.5, 72.0), turned to 90 degrees
- moved TP1 89.1 mm to (203.5, 72.0), turned to 90 degrees
- moved Q4 84.9 mm to (191.5, 83.5), turned to 90 degrees
- moved Q1 77.6 mm to (185.0, 72.0), turned to 270 degrees
- moved Q2 75.0 mm to (191.5, 72.0), turned to 90 degrees
- moved R6 74.4 mm to (194.0, 89.5)
- moved R2 73.9 mm to (194.0, 78.0)
- moved U1 73.7 mm to (169.5, 83.5), turned to 270 degrees
- moved Q3 69.1 mm to (185.0, 83.5), turned to 270 degrees
- moved C1 64.7 mm to (188.2, 78.0)
- moved C2 64.7 mm to (188.2, 89.5)
- moved R11 64.3 mm to (197.5, 95.0), turned to 90 degrees
- moved R5 63.4 mm to (180.5, 81.5), turned to 270 degrees
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Connections:
- net /Power/VCCIO renamed /Power/3V3_OUT
- U1 pad 26: (no net) -> /Power/FAULT
Other:
- board outline removed
- copper layers 2 -> 4

Commit message: wip power xESC2
Parts:
- added U4: STM32F405RGTx, Package_QFP:LQFP-64_10x10mm_P0.5mm, F.Cu at (226.2, 114.0)
- C15: value 1uF/50V -> 47uF/100V; footprint Capacitor_SMD:C_0805_2012Metric -> Capacitor_THT:CP_Radial_D8.0mm_P3.50mm
- C18: value 100uF/16V -> 1uF/50V; footprint Capacitor_SMD:CP_Elec_6.3x7.7 -> Capacitor_SMD:C_0805_2012Metric
- C19: value 10uF/25V -> 100uF/16V; footprint Capacitor_SMD:C_1206_3216Metric -> Capacitor_SMD:CP_Elec_6.3x7.7
- C21: value 47uF/100V -> 10uF/25V; footprint Capacitor_THT:CP_Radial_D8.0mm_P3.50mm -> Capacitor_SMD:C_1206_3216Metric
- TP1, TP2, TP3, TP4, TP5, TP6, TP7: footprint TestPoint:TestPoint_Pad_4.0x4.0mm -> xESC2:SolderPadHighCurrent
- moved TP6 93.7 mm to (244.8, 104.0)
- moved C6 93.5 mm to (244.1, 110.0), turned to 0 degrees
- moved TP7 92.7 mm to (244.8, 138.0), turned to 180 degrees
- moved R13 91.4 mm to (240.6, 110.0), turned to 0 degrees
- moved R14 91.0 mm to (244.1, 108.0), turned to 0 degrees
- moved C5 89.4 mm to (244.2, 112.0), turned to 180 degrees
- moved R15 88.8 mm to (240.6, 108.0), turned to 0 degrees
- moved C13 85.7 mm to (239.2, 130.8)
- moved Q5 85.3 mm to (262.8, 130.0), turned to 180 degrees
- moved Q3 85.1 mm to (262.8, 118.0), turned to 180 degrees
- moved C4 85.0 mm to (240.4, 112.0)
- moved Q1 84.9 mm to (262.8, 106.0), turned to 180 degrees
- moved C10 84.8 mm to (252.0, 128.0)
- moved C11 84.2 mm to (242.8, 128.2)
- moved R9 83.9 mm to (256.8, 128.0), turned to 180 degrees
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Connections:
- C15 pad 1: Net-(C15-Pad1) -> /VREG/VIN
- C15 pad 2: /Power/VM -> GND
- C16 pad 1: /Power/VM -> Net-(C16-Pad1)
- C16 pad 2: GND -> /VREG/VIN
- C17 pad 1: /Power/5V_OUT -> /VREG/VIN
- C18 pad 1: /Power/5V_OUT -> /VREG/5V_OUT
- C19 pad 1: /Power/5V_OUT -> /VREG/5V_OUT
- C20 pad 1: /Power/3V3_OUT -> /VREG/5V_OUT
- C21 pad 1: /Power/VM -> /VREG/3V3_OUT
- C7 pad 1: /Power/3V3_OUT -> /Power/VCCIO
- L1 pad 2: /Power/5V_OUT -> /VREG/5V_OUT
- R13 pad 1: /Power/3V3_OUT -> /Power/VCCIO
- U1 pad 19: /Power/3V3_OUT -> /Power/VCCIO
- U1 pad 25: /Power/3V3_OUT -> /Power/VCCIO
- U2 pad 1: /Power/5V_OUT -> /VREG/5V_OUT
- U2 pad 3: Net-(C15-Pad1) -> Net-(C16-Pad1)
- U2 pad 4: /Power/VM -> /VREG/VIN
- U3 pad 2: /Power/3V3_OUT -> /VREG/3V3_OUT
- U3 pad 3: /Power/5V_OUT -> /VREG/5V_OUT
Routing:
- net Net-(C25-Pad1): track 0.00 -> 32.5 mm, vias 0 -> 43
- net /Power/LSW: track 0.00 -> 32.0 mm, vias 0 -> 2
- net Net-(C26-Pad1): track 0.00 -> 27.9 mm, vias 0 -> 44
- net Net-(C24-Pad1): track 0.00 -> 27.4 mm, vias 0 -> 43
- net /Power/VCCIO: track 0.00 -> 26.2 mm, vias 0 -> 3
- net /Power/DRV_W: track 0.00 -> 23.5 mm, vias 0 -> 40
- net /Power/DRV_U: track 0.00 -> 22.1 mm, vias 0 -> 40
- net /Power/HSU: track 0.00 -> 20.8 mm, vias 0 -> 2
- net /Power/LSV: track 0.00 -> 20.1 mm, vias 0 -> 2
- net /Power/DRV_V: track 0.00 -> 18.8 mm, vias 0 -> 40
- net /Power/VM: track 0.00 -> 16.5 mm, vias 0 -> 101
- net GND: track 0.00 -> 15.2 mm, vias 0 -> 114
- net /Power/LSU: track 0.00 -> 14.6 mm, vias 0 -> 2
- net /Power/5VOUT: track 0.00 -> 13.8 mm, vias 0 -> 2
- net /Power/VOFS: track 0.00 -> 12.9 mm
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- added copper zone on B.Cu, net /Power/DRV_U
- added copper zone on F.Cu, net /Power/DRV_U
- added copper zone on B.Cu, net /Power/DRV_V
- added copper zone on F.Cu, net /Power/DRV_V
- added copper zone on B.Cu, net /Power/DRV_W
- added copper zone on F.Cu, net /Power/DRV_W
- added copper zone on B.Cu, net /Power/VM
- added copper zone on F.Cu, net /Power/VM
- added copper zone on VM, net /Power/VM
- added copper zone on B.Cu, net GND
- added copper zone on F.Cu, net GND
- added copper zone on GND, net GND
- added copper zone on B.Cu, net Net-(C24-Pad1)
- added copper zone on F.Cu, net Net-(C24-Pad1)
- added copper zone on B.Cu, net Net-(C25-Pad1)
- added copper zone on F.Cu, net Net-(C25-Pad1)
- added copper zone on B.Cu, net Net-(C26-Pad1)
- added copper zone on F.Cu, net Net-(C26-Pad1)
Other:
- board outline added: 60 x 40 mm
- net class Default: clearance 0.2 -> 0.127; trace_width 0.25 -> 0.127; via_dia 0.8 -> 0.4; via_drill 0.4 -> 0.2
- rule trace_clearance: 0.2 -> 0.127
- rule trace_min: 0.2 -> 0.127
- rule via_min_drill: 0.3 -> 0.2

Commit message: wip xESC2 logic
Parts:
- added Y1: Crystal, Crystal:Crystal_SMD_HC49-SD, F.Cu at (215.0, 116.0)
- C15: value 47uF/100V -> 100nF/100V; footprint Capacitor_THT:CP_Radial_D8.0mm_P3.50mm -> Capacitor_SMD:C_0805_2012Metric
- moved C15 122.5 mm to (227.0, 129.5)
- moved U3 120.2 mm to (229.5, 115.5), turned to 180 degrees
- moved C20 116.4 mm to (228.8, 110.5)
- moved L1 112.9 mm to (215.5, 106.5), turned to 180 degrees
- moved U2 104.7 mm to (225.5, 106.5), turned to 180 degrees
- moved C21 103.5 mm to (223.5, 116.2), turned to 270 degrees
- moved C19 102.3 mm to (205.5, 110.0), turned to 90 degrees
- moved C16 101.4 mm to (223.5, 102.5)
- moved C18 101.3 mm to (223.5, 111.8), turned to 270 degrees
- moved C17 97.1 mm to (227.5, 102.5)
- moved D1 83.1 mm to (205.5, 103.0), turned to 180 degrees
- moved C22 63.7 mm to (236.0, 133.0), turned to 270 degrees
- moved C23 39.8 mm to (236.0, 109.0), turned to 90 degrees
- moved H1 20.0 mm to (198.8, 138.2)
- moved H2 20.0 mm to (198.8, 103.8)
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Connections:
- net /VREG/5V_OUT renamed +5V
- C1 pad 1: /Power/VM -> /VREG/VIN
- C12 pad 2: /Power/VM -> /VREG/VIN
- C13 pad 1: /Power/VM -> /VREG/VIN
- C14 pad 1: /Power/VM -> /VREG/VIN
- C15 pad 1: /VREG/VIN -> (no net)
- C15 pad 2: GND -> (no net)
- C2 pad 1: /Power/VM -> /VREG/VIN
- C21 pad 1: /VREG/3V3_OUT -> +3V3
- C22 pad 1: /Power/VM -> /VREG/VIN
- C23 pad 1: /Power/VM -> /VREG/VIN
- C3 pad 1: /Power/VM -> /VREG/VIN
- C7 pad 1: /Power/VCCIO -> +3V3
- Q1 pad 5: /Power/VM -> /VREG/VIN
- Q3 pad 5: /Power/VM -> /VREG/VIN
- Q5 pad 5: /Power/VM -> /VREG/VIN
- R13 pad 1: /Power/VCCIO -> +3V3
- TP4 pad 1: /Power/VM -> /VREG/VIN
- TP5 pad 1: /Power/VM -> /VREG/VIN
- U1 pad 19: /Power/VCCIO -> +3V3
- U1 pad 25: /Power/VCCIO -> +3V3
- U1 pad 29: /Power/VM -> /VREG/VIN
- U1 pad 33: /Power/VM -> /VREG/VIN
- U3 pad 2: /VREG/3V3_OUT -> +3V3
- U4 pad 1: (no net) -> +3V3
- U4 pad 12: (no net) -> GND
- U4 pad 13: (no net) -> +3V3
- U4 pad 18: (no net) -> GND
- U4 pad 19: (no net) -> +3V3
- U4 pad 32: (no net) -> +3V3
- U4 pad 63: (no net) -> GND
- U4 pad 64: (no net) -> +3V3
Routing:
- net +5V: track 0.00 -> 38.1 mm
- net +3V3: track 0.00 -> 36.3 mm, vias 0 -> 3
- net /Power/VCCIO: track 26.2 -> 0.00 mm, vias 3 -> 0
- net /VREG/VIN: track 0.00 -> 24.5 mm, vias 0 -> 108
- net Net-(D1-Pad1): track 0.00 -> 19.8 mm
- net /Power/VM: track 16.5 -> 0.00 mm, vias 101 -> 0
- net Net-(C16-Pad1): track 0.00 -> 7.93 mm
- net /Power/VOFS: track 12.9 -> 18.9 mm
- net /Power/FAULT: track 0.00 -> 4.23 mm
- net /Power/5VOUT: track 13.8 -> 9.99 mm, vias 2 -> 0
- net /Power/LSW: track 32.0 -> 28.8 mm
- net /Power/LSU: track 14.6 -> 11.7 mm
- net /Power/HSW: track 10.8 -> 8.11 mm
- net /Power/DRV_U: track 22.1 -> 19.8 mm
- net Net-(C5-Pad2): track 4.57 -> 6.72 mm
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- added copper zone on F.Cu, net /VREG/VIN
- added copper zone on VM, net /VREG/VIN
- removed copper zone on F.Cu, net /Power/VM
- removed copper zone on VM, net /Power/VM
Other:
- board size 60 x 40 mm -> 80 x 40 mm

Commit message: wip logic
Parts:
- added C27: DNP, Capacitor_SMD:C_0603_1608Metric, F.Cu at (204.8, 155.0)
- added C28: DNP, Capacitor_SMD:C_0603_1608Metric, F.Cu at (208.8, 152.5)
- added C29: DNP, Capacitor_SMD:C_0603_1608Metric, F.Cu at (204.8, 157.5)
- added C30: DNP, Capacitor_SMD:C_0603_1608Metric, F.Cu at (208.8, 155.0)
- added C31: DNP, Capacitor_SMD:C_0603_1608Metric, F.Cu at (212.8, 152.5)
- added C32: 15pF, Capacitor_SMD:C_0603_1608Metric, F.Cu at (241.9, 157.5)
- added C33: 15pF, Capacitor_SMD:C_0603_1608Metric, F.Cu at (241.9, 155.0)
- added C34: 100nF/50V, Capacitor_SMD:C_0603_1608Metric, F.Cu at (237.9, 158.0)
- added C35: 2.2uF/50V, Capacitor_SMD:C_0805_2012Metric, F.Cu at (229.7, 158.7)
- added C36: 2.2uF/50V, Capacitor_SMD:C_0805_2012Metric, F.Cu at (234.1, 152.7)
- added C37: 100nF/50V, Capacitor_SMD:C_0603_1608Metric, F.Cu at (242.4, 152.5)
- added C38: 2.2uF/50V, Capacitor_SMD:C_0805_2012Metric, F.Cu at (229.7, 155.7)
- added C39: 2.2uF/50V, Capacitor_SMD:C_0805_2012Metric, F.Cu at (229.7, 152.7)
- added C40: 100nF/50V, Capacitor_SMD:C_0603_1608Metric, F.Cu at (237.9, 155.5)
- added C41: 100nF/50V, Capacitor_SMD:C_0603_1608Metric, F.Cu at (233.9, 158.0)
- added C42: 100nF/50V, Capacitor_SMD:C_0603_1608Metric, F.Cu at (238.4, 152.5)
- added C43: 100nF/50V, Capacitor_SMD:C_0603_1608Metric, F.Cu at (233.9, 155.5)
- added C44: 100nF/50V, Capacitor_SMD:C_0603_1608Metric, B.Cu at (260.0, 119.5)
- added R17: R, Resistor_SMD:R_0603_1608Metric, F.Cu at (216.8, 160.0)
- added R18: R, Resistor_SMD:R_0603_1608Metric, F.Cu at (220.8, 155.0)
- added R19: R, Resistor_SMD:R_0603_1608Metric, F.Cu at (216.8, 157.5)
- added R20: R, Resistor_SMD:R_0603_1608Metric, F.Cu at (212.8, 160.0)
- added R21: R, Resistor_SMD:R_0603_1608Metric, F.Cu at (220.8, 152.5)
- added R22: R, Resistor_SMD:R_0603_1608Metric, F.Cu at (216.8, 155.0)
- added R23: R, Resistor_SMD:R_0603_1608Metric, F.Cu at (212.8, 157.5)
- added R24: R, Resistor_SMD:R_0603_1608Metric, F.Cu at (208.8, 160.0)
- added R25: R, Resistor_SMD:R_0603_1608Metric, F.Cu at (204.8, 152.5)
- added R26: R, Resistor_SMD:R_0603_1608Metric, F.Cu at (216.8, 152.5)
- added R27: R, Resistor_SMD:R_0603_1608Metric, F.Cu at (212.8, 155.0)
- added R28: R, Resistor_SMD:R_0603_1608Metric, F.Cu at (208.8, 157.5)
- added R29: 10k, Resistor_SMD:R_0603_1608Metric, F.Cu at (204.8, 167.7)
- added R30: 10k NTC, Resistor_SMD:R_0603_1608Metric, B.Cu at (260.0, 117.0)
- added R31: 10k, Resistor_SMD:R_0603_1608Metric, B.Cu at (264.0, 119.5)
- C15: value 100nF/100V -> DNP; footprint Capacitor_SMD:C_0805_2012Metric -> Capacitor_SMD:C_0603_1608Metric
- moved C15 37.8 mm to (204.8, 160.0)
Connections:
- net /Power/DRV_U renamed /PHASE_U_RAW
- net /Power/DRV_V renamed /PHASE_V_RAW
- net /Power/DRV_W renamed /PHASE_W_RAW
- C15 pad 1: (no net) -> /CUR_U
- C15 pad 2: (no net) -> GND
- U1 pad 10: (no net) -> /CURV_5V
- U1 pad 11: (no net) -> /CURW_5V
- U1 pad 17: (no net) -> /MCU/UH
- U1 pad 18: (no net) -> /MCU/UL
- U1 pad 20: (no net) -> /MCU/VH
- U1 pad 21: (no net) -> /MCU/VL
- U1 pad 22: (no net) -> /MCU/WH
- U1 pad 23: (no net) -> /MCU/WL
- U1 pad 27: (no net) -> /Power/DRV_ENABLE
- U1 pad 9: (no net) -> /CURU_5V
- U4 pad 10: (no net) -> /CUR_U
- U4 pad 14: (no net) -> /PHASE_W_FILTERED
- U4 pad 15: (no net) -> /PHASE_V_FILTERED
- U4 pad 16: (no net) -> /PHASE_U_FILTERED
- U4 pad 31: (no net) -> Net-(C35-Pad2)
- U4 pad 34: (no net) -> /MCU/WL
- U4 pad 35: (no net) -> /MCU/VL
- U4 pad 36: (no net) -> /MCU/UL
- U4 pad 41: (no net) -> /MCU/UH
- U4 pad 42: (no net) -> /MCU/VH
- U4 pad 43: (no net) -> /MCU/WH
- U4 pad 47: (no net) -> Net-(C36-Pad2)
- U4 pad 48: (no net) -> +3V3
- U4 pad 5: (no net) -> Net-(C32-Pad1)
- U4 pad 6: (no net) -> Net-(C33-Pad1)
- U4 pad 60: (no net) -> GND
- U4 pad 7: (no net) -> /MCU/Reset
- U4 pad 8: (no net) -> /CUR_W
- U4 pad 9: (no net) -> /CUR_V
- Y1 pad 1: (no net) -> Net-(C32-Pad1)
- Y1 pad 2: (no net) -> Net-(C33-Pad1)
Routing:
- net /Power/LSW: track 28.8 -> 30.1 mm
- net /Power/HSU: track 20.9 -> 20.2 mm
- net /Power/LSV: track 18.7 -> 19.2 mm
- net GND: vias 118 -> 145
- added copper zone on B.Cu, net /Power/DRV_U
- added copper zone on B.Cu, net /Power/DRV_V
- added copper zone on B.Cu, net /Power/DRV_W
- removed copper zone on B.Cu, net /PHASE_U_RAW
- removed copper zone on B.Cu, net /PHASE_V_RAW
- removed copper zone on B.Cu, net /PHASE_W_RAW

Commit message: wip
Parts:
- moved R29 55.6 mm to (245.6, 130.0)
- moved C32 54.6 mm to (206.0, 116.4), turned to 180 degrees
- moved C15 50.1 mm to (235.1, 120.2), turned to 180 degrees
- moved C41 44.7 mm to (210.6, 119.8), turned to 180 degrees
- moved C34 44.4 mm to (206.4, 126.7), turned to 90 degrees
- moved C27 43.9 mm to (231.6, 120.2), turned to 180 degrees
- moved R20 42.6 mm to (231.6, 121.8), turned to 180 degrees
- moved C37 42.4 mm to (206.4, 130.0), turned to 90 degrees
- moved C33 41.2 mm to (220.1, 120.1)
- moved R17 40.9 mm to (235.1, 123.4)
- moved R28 40.3 mm to (235.1, 127.0)
- moved C29 39.7 mm to (228.1, 125.4)
- moved R24 38.2 mm to (228.1, 127.0)
- moved C28 37.6 mm to (228.1, 120.2), turned to 180 degrees
- moved C30 37.4 mm to (231.6, 125.4)
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Connections:
- C44 pad 1: /Power/TEMP -> /MCU/PCB_TEMP
- R16 pad 1: /Power/FAULT -> /MCU/FAULT
- R29 pad 1: /Power/DRV_ENABLE -> /MCU/DRV_ENABLE
- R30 pad 2: /Power/TEMP -> /MCU/PCB_TEMP
- R31 pad 1: /Power/TEMP -> /MCU/PCB_TEMP
- U1 pad 13: (no net) -> /MCU/DRV_NCS
- U1 pad 14: (no net) -> /MCU/DRV_SCK
- U1 pad 15: (no net) -> /MCU/DRV_MOSI
- U1 pad 16: (no net) -> /MCU/DRV_MISO
- U1 pad 26: /Power/FAULT -> /MCU/FAULT
- U1 pad 27: /Power/DRV_ENABLE -> /MCU/DRV_ENABLE
- U4 pad 17: (no net) -> /MCU/PCB_TEMP
- U4 pad 23: (no net) -> /MCU/TX_MOSI_EXT
- U4 pad 29: (no net) -> /MCU/TX_MOSI_EXT
- U4 pad 40: (no net) -> /MCU/DRV_NCS
- U4 pad 41: /MCU/UH -> /MCU/WH
- U4 pad 43: /MCU/WH -> /MCU/UH
- U4 pad 51: (no net) -> /MCU/DRV_SCK
- U4 pad 55: (no net) -> /MCU/DRV_MISO
- U4 pad 56: (no net) -> /MCU/DRV_MOSI
- U4 pad 57: (no net) -> /MCU/DRV_ENABLE
- U4 pad 59: (no net) -> /MCU/FAULT
Routing:
- net /MCU/DRV_ENABLE: track 0.00 -> 51.8 mm, vias 0 -> 2
- net /PHASE_U_RAW: track 19.8 -> 60.9 mm, vias 40 -> 42
- net /MCU/DRV_NCS: track 0.00 -> 40.7 mm, vias 0 -> 2
- net /MCU/DRV_MOSI: track 0.00 -> 37.1 mm, vias 0 -> 2
- net /CUR_U: track 0.00 -> 35.5 mm, vias 0 -> 2
- net /MCU/DRV_MISO: track 0.00 -> 35.2 mm, vias 0 -> 2
- net /CUR_V: track 0.00 -> 33.6 mm, vias 0 -> 2
- net /MCU/DRV_SCK: track 0.00 -> 32.9 mm, vias 0 -> 2
- net /MCU/UH: track 0.00 -> 32.3 mm, vias 0 -> 2
- net /MCU/WH: track 0.00 -> 31.6 mm, vias 0 -> 2
- net /PHASE_W_FILTERED: track 0.00 -> 31.6 mm, vias 0 -> 2
- net /MCU/UL: track 0.00 -> 31.5 mm, vias 0 -> 2
- net /PHASE_V_RAW: track 17.2 -> 46.0 mm, vias 40 -> 42
- net /CUR_W: track 0.00 -> 28.6 mm, vias 0 -> 2
- net /MCU/VL: track 0.00 -> 28.4 mm, vias 0 -> 2
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- added copper zone on B.Cu, net /PHASE_U_RAW
- added copper zone on B.Cu, net /PHASE_V_RAW
- added copper zone on B.Cu, net /PHASE_W_RAW
- added copper zone on B.Cu, net /VREG/VIN
- removed copper zone on B.Cu, net /Power/DRV_U
- removed copper zone on B.Cu, net /Power/DRV_V
- removed copper zone on B.Cu, net /Power/DRV_W
- removed copper zone on B.Cu, net /Power/VM
