File: PCB/xESC2/xESC2.kicad_pcb (KiCad board)
At the start: 4 copper layers, 80 x 40 mm, 100 parts, among them Q1 BSC026N08NS5, Q2 BSC026N08NS5, Q3 BSC026N08NS5, Q4 BSC026N08NS5, Q5 BSC026N08NS5, Q6 BSC026N08NS5, U1 TMC6200-TA, U2 XL2001, U3 AMS1117-3.3, U4 STM32F405RGTx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

Commit message: wip V2.0
Parts:
- added C45: DNP, Capacitor_SMD:C_0603_1608Metric, F.Cu at (200.9, 127.5)
- added C46: DNP, Capacitor_SMD:C_0603_1608Metric, F.Cu at (200.9, 130.9)
- added C47: DNP, Capacitor_SMD:C_0603_1608Metric, F.Cu at (200.9, 134.3)
- added D3: D_Schottky, Diode_SMD:D_SOD-123, F.Cu at (224.8, 132.6)
- added D4: LED, LED_SMD:LED_0603_1608Metric, F.Cu at (219.9, 140.2)
- added D5: LED, LED_SMD:LED_0603_1608Metric, F.Cu at (219.9, 138.4)
- added G***: LOGO, x-tech-logo:x-tech-logo, B.Cu at (208.4, 108.7)
- added J1: Conn_01x06_Male, Connector_PinHeader_2.54mm:PinHeader_1x06_P2.54mm_Vertical, F.Cu at (197.8, 121.5)
- added J2: U254-051T-4BH83-F1S, USB:XKB_U254-051T-4BH83-F1S, F.Cu at (226.1, 139.4)
- added J3: Conn_01x05_Male, Connector_PinHeader_2.54mm:PinHeader_1x05_P2.54mm_Vertical, F.Cu at (213.3, 139.5)
- added J4: Conn_01x05_Male, Connector_PinHeader_2.54mm:PinHeader_1x05_P2.54mm_Vertical, F.Cu at (197.8, 117.9)
- added J5: Conn_01x03_Male, Connector_PinHeader_2.54mm:PinHeader_1x03_P2.54mm_Vertical, F.Cu at (201.4, 120.5)
- added R32: 22R, Resistor_SMD:R_0603_1608Metric, F.Cu at (228.5, 133.5)
- added R33: R, Resistor_SMD:R_0603_1608Metric, F.Cu at (202.6, 127.5)
- added R34: R, Resistor_SMD:R_0603_1608Metric, F.Cu at (202.6, 130.9)
- added R35: R, Resistor_SMD:R_0603_1608Metric, F.Cu at (202.6, 134.3)
- added R36: R, Resistor_SMD:R_0603_1608Metric, F.Cu at (207.3, 122.2)
- added R37: 150R, Resistor_SMD:R_0603_1608Metric, F.Cu at (216.8, 140.2)
- added R38: 150R, Resistor_SMD:R_0603_1608Metric, F.Cu at (216.8, 138.4)
- added REF**: ESD-Logo_6.6x6mm_SilkScreen, Symbol:ESD-Logo_6.6x6mm_SilkScreen, B.Cu at (216.1, 108.4)
- added U5: SN65HVD232, Package_SO:SOIC-8_3.9x4.9mm_P1.27mm, F.Cu at (207.1, 117.8)
- C44: moved to F.Cu
- R30: value 10k NTC -> R; moved to F.Cu
- R31: value 10k -> 22R; moved to F.Cu
- moved C44 59.3 mm to (200.9, 124.1), turned to 90 degrees
- moved R30 57.8 mm to (202.6, 124.1), turned to 270 degrees
- moved R31 39.8 mm to (226.8, 133.5), turned to 270 degrees
- moved C32 11.3 mm to (216.7, 120.1), turned to 0 degrees
- moved Y1 4.70 mm to (219.7, 116.3)
- moved C21 4.52 mm to (228.0, 115.8)
- moved U3 4.30 mm to (233.8, 115.7)
- moved C33 2.60 mm to (222.7, 120.0)
- moved C41 2.41 mm to (213.0, 120.1), turned to 0 degrees
- moved C38 0.80 mm to (205.4, 135.8)
- moved C39 0.80 mm to (205.4, 133.7)
- moved C35 0.40 mm to (216.2, 136.6)
- moved C43 0.35 mm to (211.6, 136.5)
- moved TP1 0.15 mm to (273.4, 110.5)
- moved TP2 0.15 mm to (273.4, 121.0)
Connections:
- C44 pad 1: /MCU/PCB_TEMP -> /TEMP_MOTOR
- R30 pad 2: /MCU/PCB_TEMP -> /TEMP_MOTOR
- R31 pad 1: /MCU/PCB_TEMP -> /USB_DM
- R31 pad 2: GND -> Net-(J2-Pad2)
- U4 pad 17: /MCU/PCB_TEMP -> (no net)
- U4 pad 21: (no net) -> /MCU/SCK_EXT
- U4 pad 22: (no net) -> /MCU/MISO_EXT
- U4 pad 24: (no net) -> /TEMP_MOTOR
- U4 pad 26: (no net) -> /LED_GREEN
- U4 pad 27: (no net) -> /LED_RED
- U4 pad 30: (no net) -> /MCU/RX_NCS_EXT
- U4 pad 37: (no net) -> /HALL3
- U4 pad 38: (no net) -> /HALL2
- U4 pad 39: (no net) -> /HALL1
- U4 pad 44: (no net) -> /USB_DM
- U4 pad 45: (no net) -> /USB_DP
- U4 pad 46: (no net) -> /MCU/SWDIO
- U4 pad 49: (no net) -> /MCU/SWDCLK
- U4 pad 61: (no net) -> /MCU/CAN_RX
- U4 pad 62: (no net) -> /MCU/CAN_TX
Routing:
- net +3V3: track 38.2 -> 148.9 mm, vias 3 -> 9
- net +5V: track 38.1 -> 95.8 mm, vias 0 -> 8
- net /MCU/TX_MOSI_EXT: track 0.00 -> 39.2 mm, vias 0 -> 1
- net /MCU/MISO_EXT: track 0.00 -> 38.7 mm, vias 0 -> 1
- net /MCU/FAULT: track 4.11 -> 42.5 mm, vias 0 -> 2
- net /MCU/SCK_EXT: track 0.00 -> 34.8 mm, vias 0 -> 2
- net /MCU/RX_NCS_EXT: track 0.00 -> 34.4 mm, vias 0 -> 1
- net /HALL1: track 0.00 -> 32.7 mm, vias 0 -> 2
- net /HALL2: track 0.00 -> 31.1 mm, vias 0 -> 2
- net /TEMP_MOTOR: track 0.00 -> 28.4 mm, vias 0 -> 2
- net /MCU/SWDIO: track 0.00 -> 27.9 mm, vias 0 -> 3
- net /HALL3: track 0.00 -> 27.6 mm, vias 0 -> 2
- net /MCU/SWDCLK: track 0.00 -> 22.6 mm, vias 0 -> 3
- net /MCU/Reset: track 0.00 -> 20.9 mm, vias 0 -> 1
- net /LED_GREEN: track 0.00 -> 20.5 mm, vias 0 -> 2
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Other:
- outline, holes or cut-outs redrawn
- board text added: "CANH"
- board text added: "CANL"
- board text added: "CS"
- board text added: "GND"
- board text added: "HALL1"
- board text added: "HALL2"
- board text added: "HALL3"
- board text added: "MISO"
- board text added: "MOSI"
- board text added: "RESET"
- board text added: "SCK"
- board text added: "SWDCLK"
- board text added: "SWDIO"
- board text added: "TEMP_MOTOR"
- board text added: "V+"
- board text added: "VCC"
- board text added: "v2.0 - License CC BY-NC-SA 4.0 https://github.com/ClemensElflein/xESC"

Commit message: ordered
Routing:
- net /MCU/CAN_TX: track 5.78 -> 6.79 mm
- net +3V3: track 148.9 -> 149.5 mm
- net GND: vias 167 -> 191
