File: PCB/xESC2/xESC2.kicad_pcb (KiCad board)
At the start: 4 copper layers, 80 x 40 mm, 121 parts, among them J1 Conn_01x06_Male, J2 U254-051T-4BH83-F1S, J3 Conn_01x05_Male, J4 Conn_01x05_Male, J5 Conn_01x03_Male, Q1 BSC026N08NS5, Q2 BSC026N08NS5, Q3 BSC026N08NS5, Q4 BSC026N08NS5, Q5 BSC026N08NS5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

Commit message: changed some values, added BOM
Parts:
- C35, C36, C38, C39, C4, C5: value 2.2uF/50V -> 2.2uF/25V
- R17, R19, R21, R24, R26, R28: value R -> 1k5
- R18, R20, R22, R33, R34, R35: value R -> 2k2
- R23, R25, R27: value R -> 22k
- R30: value R -> 10k
- R36: value R -> 120R
