File: PCB/xESC2_mini/xESC2.kicad_pcb (KiCad board)
At the start: 4 copper layers, 49.5 x 29 mm, 110 parts, among them J1 Conn_01x06_Male, J10 Conn_01x06_Male, J2 U254-051T-4BH83-F1S, J3 Conn_01x05_Male, J4 Conn_01x05_Male, J5 Conn_01x03_Male, J6 Conn_02x02_Counter_Clockwise, J7 Conn_02x02_Counter_Clockwise, J8 Conn_02x02_Counter_Clockwise, J9 Conn_01x06_Male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

Commit message: Revert "wip"
This reverts commit 861f79ebd4b110dca06682843c28bd40f0364941.
Parts:
- moved G*** 63.6 mm to (213.0, 84.7)
- moved REF** 63.6 mm to (220.7, 84.4)
Routing:
- added copper zone on VM, net +3V3
- added copper zone on VM, net /VM
- added copper zone on GND, net GND
- removed copper zone on In2.Cu, net +3V3
- removed copper zone on In2.Cu, net /VM
- removed copper zone on In1.Cu, net GND
Other:
- net class Default added: clearance 0.127, trace_width 0.127, via_dia 0.4, via_drill 0.2

Commit message: wip
Parts:
- moved G*** 63.6 mm to (247.8, 137.9)
- moved REF** 63.6 mm to (255.5, 137.6)
Routing:
- added copper zone on In2.Cu, net +3V3
- added copper zone on In2.Cu, net /VM
- added copper zone on In1.Cu, net GND
- removed copper zone on VM, net +3V3
- removed copper zone on VM, net /VM
- removed copper zone on GND, net GND
Other:
- net class Default removed
