File: PCB/xESC2_mini/xESC2.sch (KiCad schematic (older format))
At the start: 44 parts, among them J1 Conn_01x06_Male, J2 U254-051T-4BH83-F1S, J3 Conn_01x05_Male, J4 Conn_01x05_Male, J5 Conn_01x03_Male, U5 SN65HVD232

Commit message: wip
Other:
- note removed: "TODO: add 5v in"
Changed lines of the file:
@@
 Text Label 3850 3900 0    50   ~ 0
 V_M_FILTERED
-Text Notes 1150 700  0    197  ~ 39
-TODO: add 5v in
 $Comp
 L Device:Thermistor_NTC TH1

Commit message: Revert "wip"
This reverts commit 861f79ebd4b110dca06682843c28bd40f0364941.
Other:
- note added: "TODO: add 5v in"
Changed lines of the file:
@@
 Text Label 3850 3900 0    50   ~ 0
 V_M_FILTERED
+Text Notes 1150 700  0    197  ~ 39
+TODO: add 5v in
 $Comp
 L Device:Thermistor_NTC TH1

Commit message: Update xESC2.sch
Other:
- note removed: "TODO: add 5v in"
Changed lines of the file:
@@
 F20 "PHASE_V" O L 8800 4150 50
 F21 "PHASE_W" O L 8800 4250 50
-F22 "TEMP" O L 8800 4400 50
 $EndSheet
 $Sheet
@@
 Text Label 3850 3900 0    50   ~ 0
 V_M_FILTERED
-Text Notes 1150 700  0    197  ~ 39
-TODO: add 5v in
 $Comp
 L Device:Thermistor_NTC TH1

Commit message: added fiducials
Parts:
- added FID1, FID2, FID3, FID4, FID5, FID6, FID7, FID8: Fiducial, Fiducial:Fiducial_0.75mm_Mask1.5mm, symbol Mechanical:Fiducial
Changed lines of the file:
@@
 Text Label 7000 4400 2    50   ~ 0
 PCB_TEMP
+$Comp
+L Mechanical:Fiducial FID1
+U 1 1 624F1524
+P 10700 3250
+F 0 "FID1" H 10785 3296 50  0000 L CNN
+F 1 "Fiducial" H 10785 3205 50  0000 L CNN
+F 2 "Fiducial:Fiducial_0.75mm_Mask1.5mm" H 10700 3250 50  0001 C CNN
+F 3 "~" H 10700 3250 50  0001 C CNN
+	1    10700 3250
+	1    0    0    -1
+$EndComp
+$Comp
+L Mechanical:Fiducial FID6
+U 1 1 624F2CC8
+P 10700 3450
+F 0 "FID6" H 10785 3496 50  0000 L CNN
+F 1 "Fiducial" H 10785 3405 50  0000 L CNN
+F 2 "Fiducial:Fiducial_0.75mm_Mask1.5mm" H 10700 3450 50  0001 C CNN
+F 3 "~" H 10700 3450 50  0001 C CNN
+	1    10700 3450
+	1    0    0    -1
+$EndComp
+$Comp
+L Mechanical:Fiducial FID7
+U 1 1 624FD30C
+P 10700 3650
+F 0 "FID7" H 10785 3696 50  0000 L CNN
+F 1 "Fiducial" H 10785 3605 50  0000 L CNN
+F 2 "Fiducial:Fiducial_0.75mm_Mask1.5mm" H 10700 3650 50  0001 C CNN
+F 3 "~" H 10700 3650 50  0001 C CNN
+	1    10700 3650
+	1    0    0    -1
+$EndComp
+$Comp
+L Mechanical:Fiducial FID8
+U 1 1 62507A8D
+P 10700 3850
+F 0 "FID8" H 10785 3896 50  0000 L CNN
+F 1 "Fiducial" H 10785 3805 50  0000 L CNN
+F 2 "Fiducial:Fiducial_0.75mm_Mask1.5mm" H 10700 3850 50  0001 C CNN
+F 3 "~" H 10700 3850 50  0001 C CNN
+	1    10700 3850
+	1    0    0    -1
+$EndComp
+$Comp
+L Mechanical:Fiducial FID2
+U 1 1 6251351C
+P 10450 3250
+F 0 "FID2" H 10535 3296 50  0000 L CNN
+F 1 "Fiducial" H 10535 3205 50  0000 L CNN
+F 2 "Fiducial:Fiducial_0.75mm_Mask1.5mm" H 10450 3250 50  0001 C CNN
+F 3 "~" H 10450 3250 50  0001 C CNN
+	1    10450 3250
+	1    0    0    -1
+$EndComp
+$Comp
+L Mechanical:Fiducial FID3
+U 1 1 62513522
+P 10450 3450
+F 0 "FID3" H 10535 3496 50  0000 L CNN
+F 1 "Fiducial" H 10535 3405 50  0000 L CNN
+F 2 "Fiducial:Fiducial_0.75mm_Mask1.5mm" H 10450 3450 50  0001 C CNN
+F 3 "~" H 10450 3450 50  0001 C CNN
+	1    10450 3450
+	1    0    0    -1
+$EndComp
+$Comp
+L Mechanical:Fiducial FID4
+U 1 1 62513528
+P 10450 3650
+F 0 "FID4" H 10535 3696 50  0000 L CNN
+F 1 "Fiducial" H 10535 3605 50  0000 L CNN
+F 2 "Fiducial:Fiducial_0.75mm_Mask1.5mm" H 10450 3650 50  0001 C CNN
+F 3 "~" H 10450 3650 50  0001 C CNN
+	1    10450 3650
+	1    0    0    -1
+$EndComp
+$Comp
+L Mechanical:Fiducial FID5
+U 1 1 6251352E
+P 10450 3850
+F 0 "FID5" H 10535 3896 50  0000 L CNN
+F 1 "Fiducial" H 10535 3805 50  0000 L CNN
+F 2 "Fiducial:Fiducial_0.75mm_Mask1.5mm" H 10450 3850 50  0001 C CNN
+F 3 "~" H 10450 3850 50  0001 C CNN
+	1    10450 3850
+	1    0    0    -1
+$EndComp
 $EndSCHEMATC
