File: PCB/xESC2_mini/Power.kicad_sch (KiCad schematic)
At the start: 20 parts, among them J10 Conn_01x06_Male, J9 Conn_01x06_Male, U1 TMC6200-TA

Commit message: wip - most routing for RP2040 done
Parts:
- C29: renamed from C6; value .1uF/100V -> .1uF
- C30: renamed from C7; value .1uF/100V -> .1uF
- C32: renamed from C12; value 100nF/100V -> .1uF; footprint Capacitor_SMD:C_0805_2012Metric -> Capacitor_SMD:C_0603_1608Metric; Digikey use the 603 in next rev -> (none)
- C33: renamed from C13; value 100nF/100V -> .1uF; footprint Capacitor_SMD:C_0805_2012Metric -> Capacitor_SMD:C_0603_1608Metric; Digikey use the 603 in next rev -> (none)
- C34: renamed from C14; value 100nF/100V -> .1uF; footprint Capacitor_SMD:C_0805_2012Metric -> Capacitor_SMD:C_0603_1608Metric; Digikey use the 603 in next rev -> (none)
- R32: renamed from R29; value 10k -> 10K
- R35: renamed from R14; value 10k -> 10K
- R36: renamed from R15; value 10k -> 10K
- renumbered C4 to C27, C5 to C28, C11 to C31, C8 to C35, C9 to C36, C10 to C37, D2 to D4, J9 to J8, J10 to J9, R16 to R33, R13 to R34, U1 to U4
