File: PCB/xESC2040/CAN.kicad_sch (KiCad schematic)
At the start: 8 parts, among them J5 Conn_01x03_Male, U1 SN65HVD232, U7 MCP2515-xST, Y2 Crystal_GND24

Commit message: added interrupt pin, added vias to the shunt, moved some stuff
Connections:
- net INT: now reaches U7.13 (~{INT})
- no-connect marks 7 -> 6
Changed lines of the file:
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@@
   (no_connect (at 162.56 104.14))
   (no_connect (at 162.56 106.68))
-  (no_connect (at 162.56 93.98))
   (no_connect (at 193.04 104.14))
   (wire (pts (xy 106.68 81.28) (xy 162.56 81.28))
@@
     (stroke (width 0) (type default) (color 0 0 0 0))
   )
+  (hierarchical_label "INT" (shape output) (at 162.56 93.98 180)
+    (effects (font (size 1.27 1.27)) (justify right))
+  )
   (hierarchical_label "MISO" (shape output) (at 193.04 81.28 0)

Commit message: Added some part numbers and such for the BoM.
Parts:
- C4, C7: Digikey (none) -> 311-1063-1-ND; Part Number (none) -> CC0603JRNPO9BN270; Stock_PN (none) -> C-603-27pF-50V-COG
- U7: Digikey (none) -> MCP2515-E/ST-ND; Part Number (none) -> MCP2515-E/ST; Stock_PN (none) -> U-MCP2515-E/ST
Changed lines of the file:
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@@
+      (effects (font (size 1.27 1.27)) hide)
+    )
+    (property "Digikey" "311-1063-1-ND" (id 4) (at 238.125 99.06 0)
+      (effects (font (size 1.27 1.27)) hide)
+    )
+    (property "Part Number" "CC0603JRNPO9BN270" (id 5) (at 238.125 99.06 0)
+      (effects (font (size 1.27 1.27)) hide)
+    )
+    (property "Stock_PN" "C-603-27pF-50V-COG" (id 6) (at 238.125 99.06 0)
       (effects (font (size 1.27 1.27)) hide)
     )
@@
     )
     (property "Datasheet" "http://ww1.microchip.com/downloads/en/DeviceDoc/21801e.pdf" (id 3) (at 175.26 114.3 0)
+      (effects (font (size 1.27 1.27)) hide)
+    )
+    (property "Digikey" "MCP2515-E/ST-ND" (id 4) (at 177.8 93.98 0)
+      (effects (font (size 1.27 1.27)) hide)
+    )
+    (property "Part Number" "MCP2515-E/ST" (id 5) (at 177.8 93.98 0)
+      (effects (font (size 1.27 1.27)) hide)
+    )
+    (property "Stock_PN" "U-MCP2515-E/ST" (id 6) (at 177.8 93.98 0)
       (effects (font (size 1.27 1.27)) hide)
     )
@@
       (effects (font (size 1.27 1.27)) hide)
     )
+    (property "Digikey" "311-1063-1-ND" (id 4) (at 238.125 106.68 0)
+      (effects (font (size 1.27 1.27)) hide)
+    )
+    (property "Part Number" "CC0603JRNPO9BN270" (id 5) (at 238.125 106.68 0)
+      (effects (font (size 1.27 1.27)) hide)
+    )
+    (property "Stock_PN" "C-603-27pF-50V-COG" (id 6) (at 238.125 106.68 0)
+      (effects (font (size 1.27 1.27)) hide)
+    )

Commit message: Added Config field for KiBoM compatability
Added Config field so with and without CAN BoM's can be generated with KiBoM
Parts:
- R4, U1, U7, Y2: Config (none) -> +can
Changed lines of the file:
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@@
+      (effects (font (size 1.27 1.27)) hide)
+    )
+    (property "Config" "+can" (id 7) (at 226.695 102.87 0)
       (effects (font (size 1.27 1.27)) hide)
     )
@@
     )
     (property "Stock_PN" "R-603-120-.1W-1%" (id 6) (at 111.76 73.025 0)
+      (effects (font (size 1.27 1.27)) hide)
+    )
+    (property "Config" "+can" (id 7) (at 111.76 73.025 0)
       (effects (font (size 1.27 1.27)) hide)
     )
@@
       (effects (font (size 1.27 1.27)) hide)
     )
+    (property "Config" "+can" (id 7) (at 177.8 93.98 0)
+      (effects (font (size 1.27 1.27)) hide)
+    )
     (pin "1")
     (pin "10")
@@
       (effects (font (size 1.27 1.27)) hide)
     )
+    (property "Config" "+can" (id 8) (at 90.17 73.025 0)
+      (effects (font (size 1.27 1.27)) hide)
+    )

Commit message: changed CAN terminator to 805 part for power handling and moved to bottom side.
Parts:
- R4: footprint Resistor_SMD:R_0603_1608Metric -> Resistor_SMD:R_0805_2012Metric; Digikey RMCF0603FT120R -> 738-RMCF0805FT120RCT-ND; Part Number RMCF0603FT120RCT-ND -> RMCF0805FT120R; Stock_PN R-603-120-.1W-1% -> R-805-120-.25W-1%
Connections:
- net CAN_P: now reaches J5.3 (Pin_3), R4.1, U1.7 (CANH)
- net CAN_N: now reaches J5.2 (Pin_2), R4.2, U1.6 (CANL)
Changed lines of the file:
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@@
     (stroke (width 0) (type default) (color 0 0 0 0))
+  )
+  (label "CAN_P" (at 104.14 69.342 0)
+    (effects (font (size 1.27 1.27)) (justify left bottom))
+  )
+  (label "CAN_N" (at 100.33 75.565 0)
+    (effects (font (size 1.27 1.27)) (justify left bottom))
   )
   (hierarchical_label "INT" (shape output) (at 162.56 93.98 180)
@@
       (effects (font (size 1.27 1.27)) (justify left))
     )
-    (property "Footprint" "Resistor_SMD:R_0603_1608Metric" (id 2) (at 109.982 73.025 90)
+    (property "Footprint" "Resistor_SMD:R_0805_2012Metric" (id 2) (at 109.982 73.025 90)
       (effects (font (size 1.27 1.27)) hide)
     )
@@
       (effects (font (size 1.27 1.27)) hide)
     )
-    (property "Digikey" "RMCF0603FT120R" (id 4) (at 111.76 73.025 0)
+    (property "Digikey" "738-RMCF0805FT120RCT-ND" (id 4) (at 111.76 73.025 0)
       (effects (font (size 1.27 1.27)) hide)
     )
-    (property "Part Number" "RMCF0603FT120RCT-ND" (id 5) (at 111.76 73.025 0)
+    (property "Part Number" "RMCF0805FT120R" (id 5) (at 111.76 73.025 0)
       (effects (font (size 1.27 1.27)) hide)
     )
-    (property "Stock_PN" "R-603-120-.1W-1%" (id 6) (at 111.76 73.025 0)
+    (property "Stock_PN" "R-805-120-.25W-1%" (id 6) (at 111.76 73.025 0)
       (effects (font (size 1.27 1.27)) hide)
     )

Commit message: add pn's for header pins - all cheapies from LSCS
Parts:
- J5: LCSC (none) -> C2935909; Part Number (none) -> DZ254R-11-03-63; Stock_PN (none) -> J-TH-1x3-.1
Changed lines of the file:
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@@
+      (effects (font (size 1.27 1.27)) hide)
+    )
+    (property "LCSC" "C2935909" (id 4) (at 124.46 71.755 0)
+      (effects (font (size 1.27 1.27)) hide)
+    )
+    (property "Part Number" "DZ254R-11-03-63" (id 5) (at 124.46 71.755 0)
+      (effects (font (size 1.27 1.27)) hide)
+    )
+    (property "Stock_PN" "J-TH-1x3-.1" (id 6) (at 124.46 71.755 0)
       (effects (font (size 1.27 1.27)) hide)
     )

Commit message: Change part for J5 to be a 9 pin header so can be soldered along with J1 to ease assembly - J1 marked as DNP
Parts:
- J5: LCSC C2935909 -> C2935915; Part Number DZ254R-11-03-63 -> DZ254R-11-09-63; Stock_PN J-TH-1x3-.1 -> J-TH-1x9-.1
Changed lines of the file:
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@@
       (effects (font (size 1.27 1.27)) hide)
     )
-    (property "LCSC" "C2935909" (id 4) (at 124.46 71.755 0)
+    (property "LCSC" "C2935915" (id 4) (at 124.46 71.755 0)
       (effects (font (size 1.27 1.27)) hide)
     )
-    (property "Part Number" "DZ254R-11-03-63" (id 5) (at 124.46 71.755 0)
+    (property "Part Number" "DZ254R-11-09-63" (id 5) (at 124.46 71.755 0)
       (effects (font (size 1.27 1.27)) hide)
     )
-    (property "Stock_PN" "J-TH-1x3-.1" (id 6) (at 124.46 71.755 0)
+    (property "Stock_PN" "J-TH-1x9-.1" (id 6) (at 124.46 71.755 0)
       (effects (font (size 1.27 1.27)) hide)
     )

Commit message: Merge J5 and J1 into one connector - no pinout changes or connector move
With J5 gone had kicad redo  reference designators - hope that's ok
Parts:
- removed J5: Conn_01x03_Male, Connector_PinHeader_2.54mm:PinHeader_1x03_P2.54mm_Vertical, symbol Connector:Conn_01x03_Male
- renumbered C4 to C28, C7 to C29, R4 to R23, R5 to R24, U1 to U6
Changed lines of the file:
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@@
 (kicad_sch (version 20211123) (generator eeschema)
   (paper "A4")
-  (junction (at 90.17 84.455) (diameter 0) (color 0 0 0 0)
-  )
   (junction (at 111.76 76.835) (diameter 0) (color 0 0 0 0)
   )
@@
     (stroke (width 0) (type default) (color 0 0 0 0))
   )
-  (wire (pts (xy 119.38 74.295) (xy 119.38 84.455))
-    (stroke (width 0) (type default) (color 0 0 0 0))
-  )
-  (wire (pts (xy 90.17 84.455) (xy 90.17 88.265))
-    (stroke (width 0) (type default) (color 0 0 0 0))
-  )
   (wire (pts (xy 74.93 55.245) (xy 107.95 55.245))
     (stroke (width 0) (type default) (color 0 0 0 0))
@@
     (stroke (width 0) (type default) (color 0 0 0 0))
   )
-  (wire (pts (xy 119.38 84.455) (xy 90.17 84.455))
-    (stroke (width 0) (type default) (color 0 0 0 0))
-  )
   (wire (pts (xy 76.2 56.515) (xy 76.2 70.485))
     (stroke (width 0) (type default) (color 0 0 0 0))
@@
     (stroke (width 0) (type default) (color 0 0 0 0))
   )
-  (wire (pts (xy 90.17 83.185) (xy 90.17 84.455))
+  (wire (pts (xy 90.17 83.185) (xy 90.17 88.265))
     (stroke (width 0) (type default) (color 0 0 0 0))
   )
@@
     (effects (font (size 1.27 1.27)) (justify right))
   )
+  (hierarchical_label "CAN_N" (shape input) (at 119.38 71.755 0)
+    (effects (font (size 1.27 1.27)) (justify left))
+  )
+  (hierarchical_label "CAN_P" (shape input) (at 119.38 69.215 0)
+    (effects (font (size 1.27 1.27)) (justify left))
+  )
   (hierarchical_label "MISO" (shape output) (at 193.04 81.28 0)
     (effects (font (size 1.27 1.27)) (justify left))
@@
   (symbol (lib_id "power:GND") (at 243.205 110.49 0) (unit 1)
     (in_bom yes) (on_board yes)
-    (property "Reference" "#PWR0107" (id 0) (at 243.205 116.84 0)
+    (property "Reference" "#PWR042" (id 0) (at 243.205 116.84 0)
       (effects (font (size 1.27 1.27)) hide)
     )
@@
   (symbol (lib_id "Device:R") (at 111.76 73.025 0) (unit 1)
     (in_bom yes) (on_board yes)
-    (property "Reference" "R4" (id 0) (at 113.538 71.8566 0)
+    (property "Reference" "R23" (id 0) (at 113.538 71.8566 0)
       (effects (font (size 1.27 1.27)) (justify left))
     )
@@
   (symbol (lib_id "Device:R_Small") (at 154.94 109.22 90) (unit 1)
     (in_bom yes) (on_board yes) (fields_autoplaced)
-    (property "Reference" "R5" (id 0) (at 154.94 104.5169 90))
+    (property "Reference" "R24" (id 0) (at 154.94 104.5169 90))
     (property "Value" "10K" (id 1) (at 154.94 107.292 90))
     (property "Footprint" "Resistor_SMD:R_0603_1608Metric" (id 2) (at 154.94 109.22 0)
@@
   (symbol (lib_id "power:GND") (at 177.8 121.92 0) (unit 1)
     (in_bom yes) (on_board yes)
-    (property "Reference" "#PWR0108" (id 0) (at 177.8 128.27 0)
+    (property "Reference" "#PWR041" (id 0) (at 177.8 128.27 0)
       (effects (font (size 1.27 1.27)) hide)
     )
@@
   (symbol (lib_id "Device:C_Small") (at 238.125 99.06 270) (unit 1)
     (in_bom yes) (on_board yes) (fields_autoplaced)
-    (property "Reference" "C4" (id 0) (at 238.1187 104.5886 90))
+    (property "Reference" "C28" (id 0) (at 238.1187 104.5886 90))
     (property "Value" "27pF" (id 1) (at 238.1187 101.8135 90))
     (property "Footprint" "Capacitor_SMD:C_0603_1608Metric" (id 2) (at 238.125 99.06 0)
@@
     (pin "1")
     (pin "2")
-  )
-  (symbol (lib_id "Connector:Conn_01x03_Male") (at 124.46 71.755 180) (unit 1)
-    (in_bom yes) (on_board yes)
-    (property "Reference" "J5" (id 0) (at 125.1712 70.0278 0)
-      (effects (font (size 1.27 1.27)) (justify right))
-    )
-    (property "Value" "Conn_01x03_Male" (id 1) (at 125.1712 72.3392 0)
-      (effects (font (size 1.27 1.27)) (justify right))
-    )
-    (property "Footprint" "Connector_PinHeader_2.54mm:PinHeader_1x03_P2.54mm_Vertical" (id 2) (at 124.46 71.755 0)
-      (effects (font (size 1.27 1.27)) hide)
-    )
-    (property "Datasheet" "~" (id 3) (at 124.46 71.755 0)
-      (effects (font (size 1.27 1.27)) hide)
-    )
-    (property "LCSC" "C2935915" (id 4) (at 124.46 71.755 0)
-      (effects (font (size 1.27 1.27)) hide)
-    )
-    (property "Part Number" "DZ254R-11-09-63" (id 5) (at 124.46 71.755 0)
-      (effects (font (size 1.27 1.27)) hide)
-    )
-    (property "Stock_PN" "J-TH-1x9-.1" (id 6) (at 124.46 71.755 0)
-      (effects (font (size 1.27 1.27)) hide)
-    )
-    (pin "1")
-    (pin "2")
-    (pin "3")
   )
   (symbol (lib_id "Interface_CAN_LIN:MCP2515-xST") (at 177.8 93.98 0) (mirror y) (unit 1)
@@
   (symbol (lib_id "Interface_CAN_LIN:SN65HVD232") (at 90.17 73.025 0) (unit 1)
     (in_bom yes) (on_board yes)
-    (property "Reference" "U1" (id 0) (at 90.17 60.8076 0))
+    (property "Reference" "U6" (id 0) (at 90.17 60.8076 0))
     (property "Value" "SN65HVD232" (id 1) (at 90.17 63.119 0))
     (property "Footprint" "Package_SO:SOIC-8_3.9x4.9mm_P1.27mm" (id 2) (at 90.17 85.725 0)
@@
   (symbol (lib_id "power:+3.3V") (at 177.8 60.325 0) (unit 1)
     (in_bom yes) (on_board yes)
-    (property "Reference" "#PWR0109" (id 0) (at 177.8 64.135 0)
+    (property "Reference" "#PWR040" (id 0) (at 177.8 64.135 0)
       (effects (font (size 1.27 1.27)) hide)
     )
@@
   (symbol (lib_id "Device:C_Small") (at 238.125 106.68 270) (unit 1)
     (in_bom yes) (on_board yes) (fields_autoplaced)
-    (property "Reference" "C7" (id 0) (at 238.1187 112.2086 90))
+    (property "Reference" "C29" (id 0) (at 238.1187 112.2086 90))
     (property "Value" "27pF" (id 1) (at 238.1187 109.4335 90))
     (property "Footprint" "Capacitor_SMD:C_0603_1608Metric" (id 2) (at 238.125 106.68 0)
@@
   (symbol (lib_id "power:+3.3V") (at 90.17 60.325 0) (unit 1)
     (in_bom yes) (on_board yes)
-    (property "Reference" "#PWR0111" (id 0) (at 90.17 64.135 0)
+    (property "Reference" "#PWR038" (id 0) (at 90.17 64.135 0)
       (effects (font (size 1.27 1.27)) hide)
     )
@@
   (symbol (lib_id "power:GND") (at 90.17 88.265 0) (unit 1)
     (in_bom yes) (on_board yes)
-    (property "Reference" "#PWR0110" (id 0) (at 90.17 94.615 0)
-      (effects (font (size 1.27 1.27)) hide)
-    )
+    (property "Reference" "#PWR039" (id 0) (at 90.17 94.615 0)
+      (effects (font (size 1.27 1.27)) hide)
+    )

Commit message: BoM data updates
Parts:
- R24: Digikey RC0603FR-0710KL -> 311-10.0KHRCT-ND; Part Number 311-10.0KHRCT-ND -> RC0603FR-0710KL
Changed lines of the file:
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@@
       (effects (font (size 1.27 1.27)) hide)
     )
-    (property "Digikey" "RC0603FR-0710KL" (id 4) (at 154.94 109.22 0)
+    (property "Digikey" "311-10.0KHRCT-ND" (id 4) (at 154.94 109.22 0)
       (effects (font (size 1.27 1.27)) hide)
     )
-    (property "Part Number" "311-10.0KHRCT-ND" (id 5) (at 154.94 109.22 0)
+    (property "Part Number" "RC0603FR-0710KL" (id 5) (at 154.94 109.22 0)
       (effects (font (size 1.27 1.27)) hide)
     )
