File: PCB/xESC2040/MCU.kicad_sch (KiCad schematic)
At the start: 20 parts, among them J5 Conn_01x02, U1 RP2040, U2 W25Q128JVP, Y1 Crystal_GND24

Commit message: wip
Parts:
- C10, C11, C12, C13, C14, C15, C16, C8, C9: Digikey 490-1331-1-ND -> 1276-1935-1-ND
- Y1: value Crystal_GND24 -> 12MHz
Changed lines of the file:
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@@
       (effects (font (size 1.27 1.27)) hide)
     )
-    (property "Digikey" "490-1331-1-ND" (id 4) (at 170.18 29.21 0)
+    (property "Digikey" "1276-1935-1-ND" (id 4) (at 170.18 29.21 0)
       (effects (font (size 1.27 1.27)) hide)
     )
@@
       (effects (font (size 1.27 1.27)) hide)
     )
-    (property "Digikey" "490-1331-1-ND" (id 4) (at 177.8 29.21 0)
+    (property "Digikey" "1276-1935-1-ND" (id 4) (at 177.8 29.21 0)
       (effects (font (size 1.27 1.27)) hide)
     )
@@
       (effects (font (size 1.27 1.27)) hide)
     )
-    (property "Digikey" "490-1331-1-ND" (id 4) (at 185.42 29.21 0)
+    (property "Digikey" "1276-1935-1-ND" (id 4) (at 185.42 29.21 0)
       (effects (font (size 1.27 1.27)) hide)
     )
@@
       (effects (font (size 1.27 1.27)) hide)
     )
-    (property "Digikey" "490-1331-1-ND" (id 4) (at 191.77 29.21 0)
+    (property "Digikey" "1276-1935-1-ND" (id 4) (at 191.77 29.21 0)
       (effects (font (size 1.27 1.27)) hide)
     )
@@
       (effects (font (size 1.27 1.27)) hide)
     )
-    (property "Digikey" "490-1331-1-ND" (id 4) (at 224.79 27.94 0)
+    (property "Digikey" "1276-1935-1-ND" (id 4) (at 224.79 27.94 0)
       (effects (font (size 1.27 1.27)) hide)
     )
@@
       (effects (font (size 1.27 1.27)) hide)
     )
-    (property "Digikey" "490-1331-1-ND" (id 4) (at 146.05 29.21 0)
+    (property "Digikey" "1276-1935-1-ND" (id 4) (at 146.05 29.21 0)
       (effects (font (size 1.27 1.27)) hide)
     )
@@
       (effects (font (size 1.27 1.27)) hide)
     )
-    (property "Digikey" "490-1331-1-ND" (id 4) (at 232.41 27.94 0)
+    (property "Digikey" "1276-1935-1-ND" (id 4) (at 232.41 27.94 0)
       (effects (font (size 1.27 1.27)) hide)
     )
@@
       (effects (font (size 1.27 1.27)) hide)
     )
-    (property "Digikey" "490-1331-1-ND" (id 4) (at 161.29 29.21 0)
+    (property "Digikey" "1276-1935-1-ND" (id 4) (at 161.29 29.21 0)
       (effects (font (size 1.27 1.27)) hide)
     )
@@
       (effects (font (size 1.27 1.27)) (justify left))
     )
-    (property "Value" "Crystal_GND24" (id 1) (at 64.008 110.6424 0)
+    (property "Value" "12MHz" (id 1) (at 64.008 110.6424 0)
       (effects (font (size 1.27 1.27)) (justify left))
     )
@@
       (effects (font (size 1.27 1.27)) hide)
     )
-    (property "Digikey" "490-1331-1-ND" (id 4) (at 153.67 29.21 0)
-      (effects (font (size 1.27 1.27)) hide)
-    )
+    (property "Digikey" "1276-1935-1-ND" (id 4) (at 153.67 29.21 0)
+      (effects (font (size 1.27 1.27)) hide)
+    )

Commit message: Update MCU.kicad_sch
Fixed part number for crystal
Parts:
- Y1: Digikey 50-ECS-80-12-33-JGN-CT-ND -> 50-ECS-120-18-33-JGN-TR3CT-ND; Part Number ECS-80-12-33-JGN-TR -> ECS-120-18-33-JGN-TR3; Stock_PN Y-4-SMD-8MhHz -> Y-1-SMD-12MhHz
Changed lines of the file:
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@@
       (effects (font (size 1.27 1.27)) hide)
     )
-    (property "Digikey" "50-ECS-80-12-33-JGN-CT-ND" (id 4) (at 62.865 115.57 0)
+    (property "Digikey" "50-ECS-120-18-33-JGN-TR3CT-ND" (id 4) (at 62.865 115.57 0)
       (effects (font (size 1.27 1.27)) hide)
     )
-    (property "Part Number" "ECS-80-12-33-JGN-TR" (id 5) (at 62.865 115.57 0)
+    (property "Part Number" "ECS-120-18-33-JGN-TR3" (id 5) (at 62.865 115.57 0)
       (effects (font (size 1.27 1.27)) hide)
     )
-    (property "Stock_PN" "Y-4-SMD-8MhHz" (id 6) (at 62.865 115.57 0)
+    (property "Stock_PN" "Y-1-SMD-12MhHz" (id 6) (at 62.865 115.57 0)
       (effects (font (size 1.27 1.27)) hide)
     )
