File: PCB/xESC2_mini_VESC/MCU.kicad_sch (KiCad schematic)
At the start: 14 parts, among them U4 STM32F405RGTx, Y1 Crystal_GND24

Commit message: updated BOM for .1uF caps
Parts:
- C34, C37, C40, C41, C42, C43: value .1uF/100V -> .1uF/50V; Digikey 490-1331-1-ND -> 1276-1935-1-ND
Changed lines of the file:
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@@
       (effects (font (size 1.27 1.27)) (justify left))
     )
-    (property "Value" ".1uF/100V" (id 1) (at 173.101 30.353 0)
+    (property "Value" ".1uF/50V" (id 1) (at 173.101 30.353 0)
       (effects (font (size 1.27 1.27)) (justify left))
     )
@@
       (effects (font (size 1.27 1.27)) hide)
     )
-    (property "Digikey" "490-1331-1-ND" (id 4) (at 170.18 29.21 0)
+    (property "Digikey" "1276-1935-1-ND" (id 4) (at 170.18 29.21 0)
       (effects (font (size 1.27 1.27)) hide)
     )
@@
       (effects (font (size 1.27 1.27)) (justify left))
     )
-    (property "Value" ".1uF/100V" (id 1) (at 180.721 30.353 0)
+    (property "Value" ".1uF/50V" (id 1) (at 180.721 30.353 0)
       (effects (font (size 1.27 1.27)) (justify left))
     )
@@
       (effects (font (size 1.27 1.27)) hide)
     )
-    (property "Digikey" "490-1331-1-ND" (id 4) (at 177.8 29.21 0)
+    (property "Digikey" "1276-1935-1-ND" (id 4) (at 177.8 29.21 0)
       (effects (font (size 1.27 1.27)) hide)
     )
@@
       (effects (font (size 1.27 1.27)) (justify left))
     )
-    (property "Value" ".1uF/100V" (id 1) (at 188.341 30.353 0)
+    (property "Value" ".1uF/50V" (id 1) (at 188.341 30.353 0)
       (effects (font (size 1.27 1.27)) (justify left))
     )
@@
       (effects (font (size 1.27 1.27)) hide)
     )
-    (property "Digikey" "490-1331-1-ND" (id 4) (at 185.42 29.21 0)
+    (property "Digikey" "1276-1935-1-ND" (id 4) (at 185.42 29.21 0)
       (effects (font (size 1.27 1.27)) hide)
     )
@@
       (effects (font (size 1.27 1.27)) (justify left))
     )
-    (property "Value" ".1uF/100V" (id 1) (at 194.691 30.353 0)
+    (property "Value" ".1uF/50V" (id 1) (at 194.691 30.353 0)
       (effects (font (size 1.27 1.27)) (justify left))
     )
@@
       (effects (font (size 1.27 1.27)) hide)
     )
-    (property "Digikey" "490-1331-1-ND" (id 4) (at 191.77 29.21 0)
+    (property "Digikey" "1276-1935-1-ND" (id 4) (at 191.77 29.21 0)
       (effects (font (size 1.27 1.27)) hide)
     )
@@
       (effects (font (size 1.27 1.27)) (justify left))
     )
-    (property "Value" ".1uF/100V" (id 1) (at 148.971 30.353 0)
+    (property "Value" ".1uF/50V" (id 1) (at 148.971 30.353 0)
       (effects (font (size 1.27 1.27)) (justify left))
     )
@@
       (effects (font (size 1.27 1.27)) hide)
     )
-    (property "Digikey" "490-1331-1-ND" (id 4) (at 146.05 29.21 0)
+    (property "Digikey" "1276-1935-1-ND" (id 4) (at 146.05 29.21 0)
       (effects (font (size 1.27 1.27)) hide)
     )
@@
       (effects (font (size 1.27 1.27)) (justify left))
     )
-    (property "Value" ".1uF/100V" (id 1) (at 36.449 47.117 0)
+    (property "Value" ".1uF/50V" (id 1) (at 36.449 47.117 0)
       (effects (font (size 1.27 1.27)) (justify left))
     )
@@
       (effects (font (size 1.27 1.27)) hide)
     )
-    (property "Digikey" "490-1331-1-ND" (id 4) (at 39.37 48.26 0)
-      (effects (font (size 1.27 1.27)) hide)
-    )
+    (property "Digikey" "1276-1935-1-ND" (id 4) (at 39.37 48.26 0)
+      (effects (font (size 1.27 1.27)) hide)
+    )
