File: PCB/xESC2_mini_VESC/VREG.kicad_sch (KiCad schematic)
At the start: 3 parts, among them U2 XC6220B331MR

Commit message: updated wrong BOM part number
Parts:
- U2: LCSC C73336 -> C86534
Changed lines of the file:
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@@
       (effects (font (size 1.27 1.27)) hide)
     )
-    (property "LCSC" "C73336" (id 6) (at 190.5 92.71 0)
+    (property "LCSC" "C86534" (id 6) (at 190.5 92.71 0)
       (effects (font (size 1.27 1.27)) hide)
     )
