File: PCB/xESC2_mini_VESC/xESC2.kicad_pcb (KiCad board)
At the start: 4 copper layers, 49.5 x 29 mm, 116 parts, among them J1 Conn_01x06_Male, J10 Conn_01x06_Male, J2 U254-051T-4BH83-F1S, J3 Conn_01x05_Male, J4 Conn_01x05_Male, J5 Conn_01x03_Male, J6 Conn_02x02_Counter_Clockwise, J7 Conn_02x02_Counter_Clockwise, J8 Conn_02x02_Counter_Clockwise, J9 Conn_01x06_Male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

Commit message: updated BOM for .1uF caps
Parts:
- C34, C37, C40, C41, C42, C43, C44, C6, C7: value 100nF/50V -> .1uF/50V
Connections:
- net /MCU/FAULT renamed /Power/FAULT
- J2 pad 4: (no net) -> unconnected-(J2-Pad4)
- U1 pad 2: (no net) -> unconnected-(U1-Pad2)
- U1 pad 28: (no net) -> unconnected-(U1-Pad28)
- U1 pad 31: (no net) -> unconnected-(U1-Pad31)
- U1 pad 35: (no net) -> unconnected-(U1-Pad35)
- U1 pad 40: (no net) -> unconnected-(U1-Pad40)
- U1 pad 45: (no net) -> unconnected-(U1-Pad45)
- U2 pad 4: (no net) -> unconnected-(U2-Pad4)
- U4 pad 2: (no net) -> unconnected-(U4-Pad2)
- U4 pad 20: (no net) -> unconnected-(U4-Pad20)
- U4 pad 25: (no net) -> unconnected-(U4-Pad25)
- U4 pad 28: (no net) -> unconnected-(U4-Pad28)
- U4 pad 3: (no net) -> unconnected-(U4-Pad3)
- U4 pad 33: (no net) -> unconnected-(U4-Pad33)
- U4 pad 4: (no net) -> unconnected-(U4-Pad4)
- U4 pad 50: (no net) -> unconnected-(U4-Pad50)
- U4 pad 52: (no net) -> unconnected-(U4-Pad52)
- U4 pad 53: (no net) -> unconnected-(U4-Pad53)
- U4 pad 54: (no net) -> unconnected-(U4-Pad54)
- U4 pad 58: (no net) -> /MCU/SERVO
- U5 pad 5: (no net) -> unconnected-(U5-Pad5)
- U5 pad 8: (no net) -> unconnected-(U5-Pad8)
Routing:
- added copper zone on In2.Cu, net +3V3
- added copper zone on In2.Cu, net /VM
- added copper zone on In1.Cu, net GND
- removed copper zone on VM, net +3V3
- removed copper zone on VM, net /VM
- removed copper zone on GND, net GND
Other:
- net class Default removed
